File: pcb/sheet1.sch (KiCad schematic (older format))
At the start: 118 parts, among them J16 Aud_Conn, J17 Main_Connector, J18 Cat_Box_Conn, J20 J20, Q1 2N3904, Y1 12.096MHz

Commit message: Continued with the schematic
Parts:
- added B_1: LS244B, symbol star_wars_arcade_main_pcb:LS244B
- added C5: .1uf, symbol Device:C
- added C_1: LS244C, symbol star_wars_arcade_main_pcb:LS244C
- added C_2: 68B09E, symbol star_wars_arcade_main_pcb:68B09E
- added D/E0, E_4: LS245A, symbol star_wars_arcade_main_pcb:LS245A
- added D_8: LS00, symbol Asteroids:LS00
- added K_2, K_6: LS08, symbol Asteroids:LS08
- added unit 2 of N_1
- added unit 4 of P_3
- added R10: 1k, symbol Device:R_US
- added R15: 10k, symbol Device:R_US
- added TPHALT, TPRW, TPRWB: TP, symbol Star_Wars_Vector_PCB:TP
Connections:
- net +5V: now also B_1.20 (VCC), C5.1, C_1.20 (VCC), C_2.7 (VCC), D/E0.20 (VCC), E_4.20 (VCC), R10.2, R15.2
- net 1.5MHZ: now also B_1.11 (I0b), D_8.5
- net 6MHZ: now also B_1.8 (I3a)
- net A0: now also C_1.17 (I3b), C_2.8 (A0)
- net A1: now also C_1.6 (I2a), C_2.9 (A1)
- net A10: now also B_1.13 (I1b), C_2.18 (A10)
- net A11: now also B_1.4 (I1a), C_2.19 (A11)
- net A12: now also B_1.2 (I0a), C_2.20 (A12)
- net A13: now also C_2.21 (A13), K_2.9
- net A14: now also C_2.22 (A14)
- net A15: now also C_2.23 (A15)
- net A2: now also C_1.4 (I1a), C_2.10 (A2)
- net A3: now also C_1.2 (I0a), C_2.11 (A3)
- net A4: now also C_1.8 (I3a), C_2.12 (A4)
- net A5: now also C_1.15 (I2b), C_2.13 (A5)
- net A6: now also C_1.13 (I1b), C_2.14 (A6)
- net A7: now also C_1.11 (I0b), C_2.15 (A7)
- net A8: now also B_1.17 (I3b), C_2.16 (A8)
- net A9: now also B_1.15 (I2b), C_2.17 (A9)
- net AB0: now also C_1.3 (O3b)
- net AB1: now also C_1.14 (O2a)
- net AB10: now also B_1.7 (O1b)
- net AB11: now also B_1.16 (O1a)
- net AB12: now also B_1.18 (O0a)
- net AB13: now also K_2.8
- net AB2: now also C_1.16 (O1a)
- net AB3: now also C_1.18 (O0a)
- net AB4: now also C_1.12 (O3a)
- net AB5: now also C_1.5 (O2b)
- net AB6: now also C_1.7 (O1b)
- net AB7: now also C_1.9 (O0b)
- net AB8: now also B_1.3 (O3b)
- net AB9: now also B_1.5 (O2b)
- net D0: now also C_2.31 (D0), D/E0.11 (B7), E_4.11 (B7)
- net D1: now also C_2.30 (D1), D/E0.12 (B6), E_4.12 (B6)
- net D2: now also C_2.29 (D2), D/E0.13 (B5), E_4.13 (B5)
- net D3: now also C_2.28 (D3), D/E0.14 (B4), E_4.14 (B4)
- net D4: now also C_2.27 (D4), D/E0.15 (B3), E_4.15 (B3)
- net D5: now also C_2.26 (D5), D/E0.16 (B2), E_4.16 (B2)
- net D6: now also C_2.25 (D6), D/E0.17 (B1), E_4.17 (B1)
- net D7: now also C_2.24 (D7), D/E0.18 (B0), E_4.18 (B0)
- net DB0: now also E_4.9 (A7)
- net DB1: now also E_4.8 (A6)
- net DB2: now also E_4.7 (A5)
- net DB3: now also E_4.6 (A4)
- net DB4: now also E_4.5 (A3)
- net DB5: now also E_4.4 (A2)
- net DB6: now also E_4.3 (A1)
- net DB7: now also E_4.2 (A0)
- net E1.5MHZ: now also B_1.9 (O0b)
- net E3MHZ: now also B_1.14 (O2a)
- net E6MHZ: now also B_1.12 (O3a)
- net ECLKQ: now also C_2.35 (Q)
- net GND: now also B_1.1 (OEa), B_1.10 (GND), B_1.19 (OEb), C5.2, C_1.1 (OEa), C_1.10 (GND), C_1.19 (OEb), C_2.1 (VSS), C_2.39 (TSC), D/E0.10 (GND), E_4.10 (GND)
- net P94: now also K_2.10
- net PD0: now also D/E0.9 (A7)
- net PD1: now also D/E0.8 (A6)
- net PD2: now also D/E0.7 (A5)
- net PD3: now also D/E0.6 (A4)
- net PD4: now also D/E0.5 (A3)
- net PD5: now also D/E0.4 (A2)
- net PD6: now also D/E0.3 (A1)
- net PD7: now also D/E0.2 (A0)
- net R~W: now also C_2.32 (R/~W), P_3.9, TPRW.1, TPRW.2
- net ~EVMEM: now also K_6.9
- net ~HALT: now also C_2.40 (HALT), R15.1, TPHALT.1, TPHALT.2
- net ~SOUND: now also K_6.10
- net at E_5.11, R4.2, TPE.1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: now also C_2.34 (E)
- net R/~WB renamed R~W~B
- net R~W~B: now also D/E0.1 (DIR), N_1.4, TPRWB.1, TPRWB.2
- new net: C_2.2 (NMI), C_2.4 (FIRQ), R10.1
- new net: E_4.19 (CE), K_6.6
- new net: D/E0.19 (CE), K_6.8
- new net 3MHZ: B_1.6 (I2a)
- new net RWB: E_4.1 (DIR)
- new net ~MBCON: K_6.5
- new net ~MBRAM: K_6.4
- new net ~R~WB: D_8.4, N_1.3, P_3.8
- new net ~WE: D_8.6
- no-connect marks 45 -> 50
Other:
- note added: "MICROPROCESSOR"

Commit message: Finished microprocessor schematic page
Parts:
- added C4: .1uf, symbol Device:C
- added CR1: 1N914, symbol Device:D
- added E_6: LS08, symbol Asteroids:LS08
- added unit 2 of M_2
- added N_11: 082, symbol Asteroids:082
- added unit 2 of N_8
- added unit 2 of P_3
- added R11, R5: 10k, symbol Device:R_US
- added R6: 100k, symbol Device:R_US
- added R7: 220, symbol Device:R_US
- added R8: 15k, symbol Device:R_US
- added R9, R97: 1k, symbol Device:R_US
- added R_10: LS14, symbol Asteroids:LS14
- added R_2: LS393A, symbol star_wars_arcade_main_pcb:LS393A
- added R_3: LS161, symbol Asteroids:LS161
- added unit 1 of R_6
- added TPRESET, TPRST1, TPRST2, TPWDDIS: TP, symbol Star_Wars_Vector_PCB:TP
Connections:
- net +10V: now also C4.1, N_11.8 (VCC), R5.2
- net +5V: now also CR1.1 (K), N_11.2 (-), R11.2, R97.1, R_2.14 (VCC), R_3.16 (VCC), R_6.14 (VCC)
- net GND: now also C4.2, N_11.4 (VSS), N_11.5 (+), N_11.6 (-), R7.1, R8.2, R_2.7 (GND), R_3.3 (A), R_3.4 (B), R_3.6 (D), R_3.8 (GND), R_6.7 (GND), TPRST1.1, TPRST1.2
- net P95: now also R_6.1 (~1CLR)
- net P96: now also M_2.10 (~1PRE_), M_2.12 (2D), R_3.10 (ET), R_3.5 (C), R_3.7 (EP)
- net ~RESET: now also C_2.37 (RESET), E_6.12, R_3.1 (C), R_6.6 (~1Q), TPRESET.1, TPRESET.2
- net at P_2.12 (2CLR), P_2.2 (1CLR): now also R_10.10, R_10.9
- net at P_2.6 (1QD): now also R_2.13 (2CK), R_3.2 (CLK)
- net at C_2.3 (IRQ): now also M_2.8 (~2Q)
- new net: N_11.1, R6.1, R7.2, R9.1
- new net: N_11.3 (+), R5.1, R6.2, R8.1
- new net: CR1.2 (A), R9.2, R_10.11, TPRST2.1, TPRST2.2
- new net: R_2.1 (1CK), R_2.8 (2QD)
- new net: N_8.6, R_2.12 (2CLR), R_2.2 (1CLR)
- new net: R_2.5 (1QC), R_6.3 (1CLK)
- new net: E_6.11, R_6.2 (1D)
- new net: E_6.13, R11.1, TPWDDIS.1, TPWDDIS.2
- new net: M_2.11 (2CLK), P_3.4, R_3.9 (LD)
- new net: P_3.3, R_3.15 (RCO)
- new net ~IRQCLR: M_2.13 (~1CLR)
- new net ~PCLR: N_8.5, R97.2, R_10.8, R_6.4 (~1PRE_)
- new net ~WDCLR: N_8.4
- no-connect marks 50 -> 63
Other:
- note added: "INTERRUPT TIMER"
- note added: "POWER-ON RESET"
- note added: "WATCHDOG"

Commit message: Added ROM to schematic
Parts:
- added E/F_2: LS244D, symbol star_wars_arcade_main_pcb:LS244D
- added F_1: 27128, symbol star_wars_arcade_main_pcb:27128
- added H/J_1, J/K_1, K/L_1, M_1: 2764, symbol star_wars_arcade_main_pcb:2764
- added unit 4 of K_2
- added unit 3 of M_3
- added R12: 10k, symbol Device:R_US
- added TPROM0, TPROM1, TPROM2, TPROM3, TPROM4: TP, symbol Star_Wars_Vector_PCB:TP
- gave numbers to parts that had none: 1
- renumbered TP+10.3UN to TP+10.3UN1, TP+12V to TP+12V1, TP-5V to TP-5V1, TP3MHZ to TP3MHZ1, TP6MHZ to TP6MHZ1, TPCATSTR to TPCATSTR1, TPE to TPE1, TPHALT to TPHALT1, TPQ to TPQ1, TPRESET to TPRESET1, TPRW to TPRW1, TPRWB to TPRWB1, TPWDDIS to TPWDDIS1
Connections:
- net +5V: now also E/F_2.20 (VCC), F_1.1 (VPP), F_1.27 (PGM), F_1.28 (VCC), H/J_1.1 (VPP), H/J_1.26 (NC), H/J_1.27 (PGM), H/J_1.28 (VCC), J/K_1.1 (VPP), J/K_1.26 (NC), J/K_1.27 (PGM), J/K_1.28 (VCC), K/L_1.1 (VPP), K/L_1.26 (NC), K/L_1.27 (PGM), K/L_1.28 (VCC), M_1.1 (VPP), M_1.26 (NC), M_1.27 (PGM), M_1.28 (VCC), R12.2
- net A15: now also M_3.9
- net D0: now also E/F_2.18 (O0a)
- net D1: now also E/F_2.16 (O1a)
- net D2: now also E/F_2.12 (O3a)
- net D3: now also E/F_2.3 (O3b)
- net D4: now also E/F_2.5 (O2b)
- net D5: now also E/F_2.14 (O2a)
- net D6: now also E/F_2.7 (O1b)
- net D7: now also E/F_2.9 (O0b)
- net GND: now also E/F_2.10 (GND), F_1.14 (GND), F_1.22 (~OE), H/J_1.14 (GND), H/J_1.22 (~OE), J/K_1.14 (GND), J/K_1.22 (~OE), K/L_1.14 (GND), K/L_1.22 (~OE), M_1.14 (GND), M_1.22 (~OE)
- new net: E/F_2.2 (I0a), F_1.11 (D0), H/J_1.11 (D0), J/K_1.11 (D0), K/L_1.11 (D0), M_1.11 (D0)
- new net: E/F_2.4 (I1a), F_1.12 (D1), H/J_1.12 (D1), J/K_1.12 (D1), K/L_1.12 (D1), M_1.12 (D1)
- new net: E/F_2.8 (I3a), F_1.13 (D2), H/J_1.13 (D2), J/K_1.13 (D2), K/L_1.13 (D2), M_1.13 (D2)
- new net: E/F_2.17 (I3b), F_1.15 (D3), H/J_1.15 (D3), J/K_1.15 (D3), K/L_1.15 (D3), M_1.15 (D3)
- new net: E/F_2.15 (I2b), F_1.16 (D4), H/J_1.16 (D4), J/K_1.16 (D4), K/L_1.16 (D4), M_1.16 (D4)
- new net: E/F_2.6 (I2a), F_1.17 (D5), H/J_1.17 (D5), J/K_1.17 (D5), K/L_1.17 (D5), M_1.17 (D5)
- new net: E/F_2.13 (I1b), F_1.18 (D6), H/J_1.18 (D6), J/K_1.18 (D6), K/L_1.18 (D6), M_1.18 (D6)
- new net: E/F_2.11 (I0b), F_1.19 (D7), H/J_1.19 (D7), J/K_1.19 (D7), K/L_1.19 (D7), M_1.19 (D7)
- new net: E/F_2.1 (OEa), E/F_2.19 (OEb), K_2.11
- new net: M_3.10, R12.1
- new net: K_2.12, M_3.8
- new net AB: F_1.10 (A0), F_1.2 (A12), F_1.21 (A10), F_1.23 (A11), F_1.24 (A9), F_1.25 (A8), F_1.3 (A7), F_1.4 (A6), F_1.5 (A5), F_1.6 (A4), F_1.7 (A3), F_1.8 (A2), F_1.9 (A1), H/J_1.10 (A0), H/J_1.2 (A12), H/J_1.21 (A10), H/J_1.23 (A11), H/J_1.24 (A9), H/J_1.25 (A8), H/J_1.3 (A7), H/J_1.4 (A6), H/J_1.5 (A5), H/J_1.6 (A4), H/J_1.7 (A3), H/J_1.8 (A2), H/J_1.9 (A1), J/K_1.10 (A0), J/K_1.2 (A12), J/K_1.21 (A10), J/K_1.23 (A11), J/K_1.24 (A9), J/K_1.25 (A8), J/K_1.3 (A7), J/K_1.4 (A6), J/K_1.5 (A5), J/K_1.6 (A4), J/K_1.7 (A3), J/K_1.8 (A2), J/K_1.9 (A1), K/L_1.10 (A0), K/L_1.2 (A12), K/L_1.21 (A10), K/L_1.23 (A11), K/L_1.24 (A9), K/L_1.25 (A8), K/L_1.3 (A7), K/L_1.4 (A6), K/L_1.5 (A5), K/L_1.6 (A4), K/L_1.7 (A3), K/L_1.8 (A2), K/L_1.9 (A1), M_1.10 (A0), M_1.2 (A12), M_1.21 (A10), M_1.23 (A11), M_1.24 (A9), M_1.25 (A8), M_1.3 (A7), M_1.4 (A6), M_1.5 (A5), M_1.6 (A4), M_1.7 (A3), M_1.8 (A2), M_1.9 (A1)
- new net MPAGE: F_1.26 (MPAGE)
- new net ~ROM0: F_1.20 (~CE), K_2.13, TPROM0.1, TPROM0.2
- new net ~ROM1: H/J_1.20 (~CE), TPROM1.1, TPROM1.2
- new net ~ROM2: J/K_1.20 (~CE), TPROM2.1, TPROM2.2
- new net ~ROM3: K/L_1.20 (~CE), TPROM3.1, TPROM3.2
- new net ~ROM4: M_1.20 (~CE), TPROM4.1, TPROM4.2
Other:
- note added: "ROM"
- moved on the sheet: B_1, C1, C2, C3, C4, C5, CR1, C_1, C_2, D/E0, D_8B, E_4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

Commit message: Added RAM to the schematic
Parts:
- added C94: 4.7uf, symbol Device:CP1
- added C95: .1uf, symbol Device:C
- added CR3: 1N914, symbol Device:D
- added E_1: x2212, symbol star_wars_arcade_main_pcb:x2212
- added F/H_2: 137211, symbol star_wars_arcade_main_pcb:137211
- added unit 2 of K_2
- added unit 4 of K_6
- added unit 1 of K_6
- added L_10: 7407, symbol Star_Wars_Vector_PCB:74LS07
- added L_8, M_8: LS138, symbol star_wars_arcade_main_pcb:LS138
- added R100: 22k, symbol Device:R_US
- added R59: 10k, symbol Device:R_US
Connections:
- net +5EAROM: now also C95.2, CR3.1 (K), E_1.18 (VCC), R100.1
- net +5V: now also F/H_2.24 (VCC), K_6.14 (VCC), L_10.14 (VCC), L_8.16 (VCC), M_8.16 (VCC)
- net AB0: now also E_1.6 (A0), F/H_2.8 (AB0)
- net AB1: now also E_1.5 (A1), F/H_2.7 (AB1)
- net AB10: now also F/H_2.19 (AB10)
- net AB2: now also E_1.4 (A2), F/H_2.6 (AB2)
- net AB3: now also E_1.3 (A3), F/H_2.5 (AB3)
- net AB4: now also E_1.2 (A4), F/H_2.4 (AB4)
- net AB5: now also E_1.16 (A5), F/H_2.3 (AB5), L_8.1 (A), M_8.1 (A)
- net AB6: now also E_1.17 (A6), F/H_2.2 (AB6), L_8.2 (B), M_8.2 (B)
- net AB7: now also E_1.1 (A7), F/H_2.1 (AB7), L_8.3 (C), M_8.3 (C)
- net AB8: now also F/H_2.23 (AB8)
- net AB9: now also F/H_2.22 (AB9)
- net D0: now also E_1.12 (IO1), F/H_2.9 (D0)
- net D1: now also E_1.13 (IO2), F/H_2.10 (D1)
- net D2: now also E_1.14 (IO3), F/H_2.11 (D2)
- net D3: now also E_1.15 (IO4), F/H_2.13 (D3)
- net D4: now also F/H_2.14 (GND)
- net D5: now also F/H_2.15 (D5)
- net D6: now also F/H_2.16 (D6)
- net D7: now also F/H_2.17 (D7)
- net GND: now also C94.2, C95.1, E_1.8 (VSS), F/H_2.14 (GND), K_6.7 (GND), L_10.7 (GND), L_8.8 (GND), M_8.8 (GND)
- net P94: now also L_8.6 (G1), M_8.6 (G1)
- net ~EVGGO: now also M_8.15 (Y0)
- net ~EVGRST: now also K_2.6
- net ~IRQCLR: now also M_8.12 (Y3)
- net ~PCLR: now also K_6.13
- net ~RESET: now also K_2.4, K_6.1
- net ~R~WB: now also F/H_2.20 (OE)
- net ~SOUNDRST: now also K_6.3
- net ~WDCLR: now also M_8.13 (Y2)
- net ~WE: now also E_1.11 (~WE), F/H_2.21 (~WE), M_8.5 (~G2B)
- new net: E_1.10 (~RC), L_10.2, R59.1
- new net: C94.1, CR3.2 (A), R100.2, R59.2
- new net: K_6.12, M_8.10 (Y5)
- new net: K_2.5, M_8.14 (Y1)
- new net: K_6.2, M_8.7 (Y7)
- new net ~ADC: L_8.11 (Y4)
- new net ~ADCSTART: M_8.9 (Y6)
- new net ~IN0: L_8.15 (Y0)
- new net ~IN1: L_8.14 (Y1)
- new net ~NOVRAM: E_1.7 (~CS)
- new net ~NSTORE: E_1.9 (~STR), K_6.11
- new net ~OLATCH: M_8.11 (Y4)
- new net ~OPT0: L_8.13 (Y2)
- new net ~OPT1: L_8.12 (Y3)
- new net ~OUTS: M_8.4 (~G2A)
- new net ~RAM: F/H_2.18 (CE)
- new net ~RECALL: L_10.1
- new net ~SW: L_8.4 (~G2A), L_8.5 (~G2B)
- no-connect marks 63 -> 66
Other:
- note added: "NON_VOLATILE RAM"
- note added: "RAM"

Commit message: Continued work on the schematic
Parts:
- added B/C_0, L_2, N_7: LS138, symbol star_wars_arcade_main_pcb:LS138
- added C7, C8: .1uf, symbol Device:C
- added CR4, CR5, CR6: BLUE LED, symbol Device:LED
- added unit 1 of D_8
- added unit 3 of E_6
- added J_2: LS139, symbol Asteroids:LS139
- added unit 1 of K_2
- added K_8: LS04, symbol Asteroids:LS04
- added L/M_9: LS259, symbol Asteroids:LS259
- added unit 2 of L_10
- added unit 3 of L_10
- added L_11: SW_DIP_x04, symbol Switch:SW_DIP_x04
- added unit 2 of M_3
- added unit 4 of N_8
- added unit 6 of P_3
- added Q3, Q4: Q_NPN_BCE, symbol Device:Q_NPN_BCE
- added R13, R14, R16, R17, R58: 1k, symbol Device:R_US
- added TPEVMEM1, TPMPAGE1: TP, symbol Star_Wars_Vector_PCB:TP
Connections:
- net +5V: now also B/C_0.16 (VCC), CR4.2 (A), CR5.2 (A), CR6.2 (A), D_8.14 (VCC), J_2.16 (VCC), K_2.14 (VCC), L/M_9.16 (VCC), L_2.16 (VCC), N_7.16 (VCC), R16.2, R17.2
- net 1.5MHZ: now also M_3.4
- net AB0: now also L/M_9.1 (A), N_7.1 (A)
- net AB1: now also J_2.13 (2B), L/M_9.2 (B), N_7.2 (B)
- net AB10: now also L_2.3 (C)
- net AB11: now also J_2.2 (1A)
- net AB12: now also J_2.3 (1B)
- net AB13: now also B/C_0.1 (A)
- net AB2: now also L/M_9.3 (C), N_7.3 (C)
- net AB8: now also L_2.1 (A)
- net AB9: now also L_2.2 (B)
- net COIN_CNTR_1: now also C7.1, L_11.1, Q3.2 (C)
- net COIN_CNTR_2: now also C8.1, L_11.8, Q4.2 (C)
- net D7: now also L/M_9.13 (D)
- net GND: now also B/C_0.4 (~G2A), B/C_0.5 (~G2B), B/C_0.8 (GND), C7.2, C8.2, D_8.7 (GND), J_2.8 (GND), K_2.7 (GND), L/M_9.8 (GND), L_2.8 (GND), N_7.8 (GND), Q3.3 (E), Q4.3 (E)
- net LED1: now also CR4.1 (K), R13.1
- net MPAGE: now also L/M_9.9 (Q4), TPMPAGE1.1, TPMPAGE1.2
- net P92: now also B/C_0.6 (G1)
- net P94: now also L_2.6 (G1)
- net P95: now also N_7.6 (G1)
- net R~W~B: now also N_8.12
- net ~DVDDH: now also N_7.9 (Y6)
- net ~DVDDL: now also N_7.7 (Y7)
- net ~DVSRH: now also N_7.11 (Y4)
- net ~DVSRL: now also N_7.10 (Y5)
- net ~EVMEM: now also E_6.8, TPEVMEM1.1, TPEVMEM1.2
- net ~MBCON: now also K_8.11, L_2.7 (Y7), N_7.5 (~G2B)
- net ~MBRAM: now also K_2.3
- net ~NOVRAM: now also L_2.10 (Y5)
- net ~OLATCH: now also L/M_9.14 (G)
- net ~OUTS: now also L_2.9 (Y6)
- net ~RAM: now also J_2.5 (1Y1)
- net ~RECALL: now also D_8.3
- net ~REH: now also J_2.12 (2Y0)
- net ~REL: now also J_2.11 (2Y1)
- net ~RESET: now also L/M_9.15 (C)
- net ~ROM0: now also B/C_0.12 (Y3)
- net ~ROM1: now also B/C_0.11 (Y4)
- net ~ROM2: now also B/C_0.10 (Y5)
- net ~ROM3: now also B/C_0.9 (Y6)
- net ~ROM4: now also B/C_0.7 (Y7)
- net ~SOUND: now also M_3.6
- net ~SW: now also L_2.12 (Y3)
- net ~WE: now also N_7.4 (~G2A)
- new net: B/C_0.13 (Y2), J_2.1 (1G)
- new net: B/C_0.14 (Y1), E_6.9
- new net: B/C_0.15 (Y0), E_6.10
- new net: J_2.4 (1Y0), L_2.4 (~G2A), L_2.5 (~G2B)
- new net: J_2.6 (1Y2), K_2.2
- new net: J_2.7 (1Y3), K_2.1
- new net: L_2.11 (Y4), P_3.13
- new net: M_3.5, P_3.12
- new net: J_2.15 (2G), N_8.11
- new net: K_8.10, N_8.13
- new net: L/M_9.11 (Q6), R13.2
- new net: D_8.1, D_8.2, L/M_9.12 (Q7)
- new net: L/M_9.4 (Q0), L_10.5, R16.1
- new net: L/M_9.5 (Q1), L_10.3, R17.1
- new net: L/M_9.6 (Q2), R58.2
- new net: L/M_9.7 (Q3), R14.2
- new net: CR5.1 (K), R14.1
- new net: CR6.1 (K), R58.1
- new net: L_10.4, Q3.1 (B)
- new net: L_10.6, Q4.1 (B)
- new net AB14: B/C_0.2 (B)
- new net AB15: B/C_0.3 (C)
- new net ~AB0: J_2.14 (2A)
- new net ~MW0: N_7.15 (Y0)
- new net ~MW1: N_7.14 (Y1)
- new net ~MW2: N_7.13 (Y2)
- new net ~PRNG: J_2.9 (2Y3)
- new net ~PRNGCLR: L/M_9.10 (Q5)
- no-connect marks 66 -> 77
Other:
- note added: "ADDRESS DECODERS"
- note added: "COIN DOOR OUTPUT"
- note added: "MATH ADDRESS DECODERS"
- note added: "TEST AND CONTROL SIGNALS"
- moved on the sheet: K_2B, K_6A, K_6D, L_8, M_8

Commit message: Worked on the schematic
Parts:
- added B_5: LS86, symbol Asteroids:LS86
- added C10, C11, C12, C13, C14, C15, C16, C17, C18, C19, C20, C45, C46, C47, C48, C9: .1uf, symbol Device:C
- added C_5, D_5: LS164A, symbol star_wars_arcade_main_pcb:LS164A
- added D_4: LS299, symbol star_wars_arcade_main_pcb:LS299
- added E_9, F_9: LS244, symbol Asteroids:LS244
- added H_9: LS244E, symbol star_wars_arcade_main_pcb:LS244E
- added J_9: LS244F, symbol star_wars_arcade_main_pcb:LS244F
- added unit 3 of K_8
- added unit 2 of K_8
- added K_9: ADC, symbol star_wars_arcade_main_pcb:ADC
- added R18, R19, R20, R21, R26, R27, R28, R29, R30, R31, R32, R33: 470, symbol Device:R_US
- added R22, R23, R24, R25, R34, R35, R36, R37, R38, R39, R40, R41: 1k, symbol Device:R_US
- added R42, R43, R44, R45, R46, R47, R48, R49, R50, R51, R52, R53, R54, R55, R56, R57: 10k, symbol Device:R_US
- added R79, R80, R81: 100, symbol Device:R_US
- added R82, R83, R84, R85, R86: 4.7k, symbol Device:R_US
- added SW3: E/F_10, symbol Switch:SW_DIP_x08
- added SW4: D_10, symbol Switch:SW_DIP_x08
- added TPCOINL1, TPCOINR1, TPCOIN_AUX1, TPDIAGN1, TPFIRE/START1, TPSELF_TEST1, TPSLAM1: TP, symbol Star_Wars_Vector_PCB:TP
Connections:
- net +5V: now also B_5.14 (VCC), C45.1, C_5.14 (VCC), D_4.20 (VCC), D_5.14 (VCC), E_9.20 (VCC), F_9.20 (VCC), H_9.20 (VCC), J_9.20 (VCC), K_9.11 (VCC), K_9.12 (REF+), R18.1, R19.1, R20.1, R21.1, R26.1, R27.1, R28.1, R29.1, R30.1, R31.1, R32.1, R33.1, R42.1, R43.1, R44.1, R45.1, R46.1, R47.1, R48.1, R49.1, R50.1, R51.1, R52.1, R53.1, R54.1, R55.1, R56.1, R57.1, R82.1, R83.1, R84.1, R85.1, R86.1
- net 3MHZ: now also C_5.8 (CLK), D_4.12 (CK~), D_5.8 (CLK)
- net 750KHZ: now also K_9.10 (CLK), R85.2
- net AB0: now also R83.2
- net AB1: now also K_9.24 (ADDB), R82.2
- net COIN_AUX: now also R32.2, R39.2
- net COIN_L: now also R31.2, R40.2
- net COIN_R: now also R30.2, R41.2
- net D0: now also D_4.16 (H~), E_9.3 (O3b), F_9.3 (O3b), H_9.7 (O1b), J_9.3 (O3b), K_9.21 (D7)
- net D1: now also D_4.4 (G~), E_9.5 (O2b), F_9.5 (O2b), H_9.16 (O1a), J_9.5 (O2b), K_9.20 (D6)
- net D2: now also D_4.15 (F~), E_9.7 (O1b), F_9.7 (O1b), H_9.18 (O0a), J_9.7 (O1b), K_9.19 (D5)
- net D3: now also D_4.5 (E~), E_9.9 (O0b), F_9.9 (O0b), H_9.3 (O3b), J_9.16 (O1a), K_9.18 (D4)
- net D4: now also D_4.14 (D~), E_9.12 (O3a), F_9.12 (O3a), H_9.9 (O0b), J_9.12 (O3a), K_9.8 (D3)
- net D5: now also D_4.6 (C~), E_9.14 (O2a), F_9.14 (O2a), H_9.12 (O3a), J_9.14 (O2a), K_9.15 (D2)
- net D6: now also D_4.13 (B~), E_9.16 (O1a), F_9.16 (O1a), H_9.14 (O2a), J_9.9 (O0b), K_9.14 (D1)
- net D7: now also D_4.7 (A~), E_9.18 (O0a), F_9.18 (O0a), H_9.5 (O2b), J_9.18 (O0a), K_9.17 (D0)
- net DIAGN: now also R18.2, R25.2
- net GND: now also B_5.7 (GND), C10.2, C11.2, C12.2, C13.2, C14.2, C15.2, C16.2, C17.2, C18.2, C19.2, C20.2, C45.2, C46.2, C47.2, C48.2, C9.2, C_5.7 (GND), D_4.10 (GND), D_4.19 (S1~), D_5.7 (GND), E_9.10 (GND), F_9.10 (GND), H_9.10 (GND), J_9.10 (GND), K_9.1 (IN3), K_9.13 (GND), K_9.16 (GND), K_9.2 (IN4), K_9.23 (ADDC), K_9.3 (IN5), K_9.4 (IN6), K_9.5 (IN7), SW3.10, SW3.11, SW3.12, SW3.13, SW3.14, SW3.15, SW3.16, SW3.9, SW4.10, SW4.11, SW4.12, SW4.13, SW4.14, SW4.15, SW4.16, SW4.9
- net L_FIRE: now also R29.2, R34.2
- net L_THUMB: now also R21.2, R22.2
- net P92: now also B_5.5, D_4.1 (S0~), D_4.18 (SL)
- net R_FIRE: now also R28.2, R35.2
- net R_THUMB: now also R20.2, R23.2
- net SELF_TEST: now also R26.2, R37.2
- net SLAM: now also R33.2, R38.2
- net SPARE1: now also R27.2, R36.2
- net SPARE2: now also R19.2, R24.2
- net VGHALT: now also H_9.6 (I2a)
- net ~ADC: now also K_8.3
- net ~ADCSTART: now also K_8.5
- net ~IN0: now also J_9.1 (OEa), J_9.19 (OEb)
- net ~IN1: now also H_9.1 (OEa), H_9.19 (OEb)
- net ~OPT0: now also E_9.1 (OEa), E_9.19 (OEb)
- net ~OPT1: now also F_9.1 (OEa), F_9.19 (OEb)
- net ~PRNG: now also D_4.2 (G1~), D_4.3 (G2~)
- net ~PRNGCLR: now also C_5.9 (C), D_4.9 (CLR~), D_5.9 (C)
- net ~THRUST: now also R79.2, R81.2
- net ~YAW: now also R80.2
- new net: C12.1, H_9.8 (I3a), R22.1
- new net: C11.1, H_9.11 (I0b), R23.1
- new net: C10.1, H_9.17 (I3b), R24.1
- new net: C9.1, H_9.2 (I0a), R25.1, TPDIAGN1.1, TPDIAGN1.2
- new net: C13.1, J_9.2 (I0a), R34.1, TPFIRE/START1.1, TPFIRE/START1.2
- new net: C14.1, J_9.11 (I0b), R35.1
- new net: C15.1, J_9.6 (I2a), R36.1
- new net: C16.1, J_9.8 (I3a), R37.1, TPSELF_TEST1.1, TPSELF_TEST1.2
- new net: C20.1, J_9.4 (I1a), R38.1, TPSLAM1.1, TPSLAM1.2
- new net: C19.1, J_9.13 (I1b), R39.1, TPCOIN_AUX1.1, TPCOIN_AUX1.2
- new net: C18.1, J_9.15 (I2b), R40.1, TPCOINL1.1, TPCOINL1.2
- new net: C17.1, J_9.17 (I3b), R41.1, TPCOINR1.1, TPCOINR1.2
- new net: F_9.11 (I0b), R53.2, SW3.4
- new net: F_9.13 (I1b), R52.2, SW3.3
- new net: F_9.15 (I2b), R51.2, SW3.2
- new net: F_9.17 (I3b), R50.2, SW3.1
- new net: F_9.2 (I0a), R57.2, SW3.8
- new net: F_9.4 (I1a), R56.2, SW3.7
- new net: F_9.6 (I2a), R55.2, SW3.6
- new net: F_9.8 (I3a), R54.2, SW3.5
- new net: E_9.11 (I0b), R45.2, SW4.4
- new net: E_9.13 (I1b), R44.2, SW4.3
- new net: E_9.15 (I2b), R43.2, SW4.2
- new net: E_9.17 (I3b), R42.2, SW4.1
- new net: E_9.2 (I0a), R49.2, SW4.8
- new net: E_9.4 (I1a), R48.2, SW4.7
- new net: E_9.6 (I2a), R47.2, SW4.6
- new net: E_9.8 (I3a), R46.2, SW4.5
- new net: B_5.6, C_5.1 (A), C_5.2 (B)
- new net: B_5.1, C_5.10 (QE)
- new net: C_5.13 (QH), D_4.11 (SR~)
- new net: D_4.17 (QH), D_5.1 (A), D_5.2 (B)
- new net: B_5.2, D_5.12 (QG)
- new net: B_5.3, B_5.4
- new net: K_8.6, K_9.22 (ALE), K_9.6 (START), R84.2
- new net: C46.1, K_9.26 (IN0), R79.1
- new net: C47.1, K_9.27 (IN1), R80.1
- new net: C48.1, K_9.28 (IN2), R81.1
- new net: K_8.4, K_9.9 (OE), R86.2
- new net MATH_RUN: H_9.15 (I2b)
- no-connect marks 77 -> 94
Other:
- note added: "ANALOG/DIGITAL CONVERTER"
- note added: "COIN DOOR AND\nCONTROL PANEL INPUT"
- note added: "OPTION SWITCHES"
- note added: "PSEUDO-RANDOM\nNUMBER GENERATOR"
- moved on the sheet: J_4, J_5, K_4, K_5, L_4, L_5, L_6, M_3A, M_3D, M_4, M_5, M_6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
