File: pcb/sheet1.sch (KiCad schematic (older format))
At the start: 275 parts, among them J16 Aud_Conn, J17 Main_Connector, J18 Cat_Box_Conn, J20 J20, Q1 2N3904, Q3 Q_NPN_BCE, Q4 Q_NPN_BCE, SW3 E/F_10, SW4 D_10, Y1 12.096MHz

Commit message: Worked on the mathbox schematic
Parts:
- added A_9, B_9: LS164A, symbol star_wars_arcade_main_pcb:LS164A
- added B_8: LS385, symbol star_wars_arcade_main_pcb:LS385
- added D_6, D_7: LS299, symbol star_wars_arcade_main_pcb:LS299
- added unit 3 of D_8
- added unit 2 of E_5
- added unit 1 of E_6
- added E_7, F_7: LS00, symbol Asteroids:LS00
- added F_5, H_5: RAM, symbol star_wars_arcade_main_pcb:RAM
- added F_6, J_3, K_3: LS153A, symbol star_wars_arcade_main_pcb:LS153A
- added H_3: LS157A, symbol star_wars_arcade_main_pcb:LS157A
- added H_7, J_7, K_7, L_7: PROM, symbol star_wars_arcade_main_pcb:PROM
- added unit 4 of K_8
- added L_3: LS157B, symbol star_wars_arcade_main_pcb:LS157B
Connections:
- net +5V: now also A_9.14 (VCC), B_8.20 (VCC), B_9.14 (VCC), D_6.20 (VCC), D_7.20 (VCC), E_6.14 (VCC), E_7.14 (VCC), F_5.24 (VCC), F_6.16 (VCC), F_7.14 (VCC), H_3.16 (VCC), H_5.24 (VCC), H_7.18 (VCC), J_3.16 (VCC), J_7.18 (VCC), K_3.16 (VCC), K_7.18 (VCC), L_3.16 (VCC), L_7.18 (VCC)
- net AB1: now also L_3.14 (4A)
- net AB10: now also H_3.5 (2A)
- net AB11: now also H_3.11 (3A)
- net AB2: now also L_3.2 (1A)
- net AB3: now also J_3.10 (2C0)
- net AB4: now also K_3.10 (2C0)
- net AB5: now also J_3.6 (1C0)
- net AB6: now also K_3.6 (1C0)
- net AB7: now also F_6.6 (1C0)
- net AB8: now also H_3.14 (4A)
- net AB9: now also H_3.2 (1A)
- net GND: now also A_9.7 (GND), B_8.10 (GND), B_8.8 (2S/~A), B_9.7 (GND), D_6.10 (GND), D_7.10 (GND), E_6.7 (GND), E_7.7 (GND), F_5.10 (~OE), F_5.12 (GND), F_5.18 (~CE), F_6.1 (~1G), F_6.15 (~2G), F_6.8 (GND), F_7.7 (GND), H_3.8 (GND), H_5.10 (~OE), H_5.12 (GND), H_5.18 (~CE), H_7.10 (~CE2), H_7.8 (~CE1), H_7.9 (GND), J_3.1 (~1G), J_3.15 (~2G), J_3.8 (GND), J_7.10 (~CE2), J_7.8 (~CE1), J_7.9 (GND), K_3.1 (~1G), K_3.15 (~2G), K_3.8 (GND), K_7.10 (~CE2), K_7.8 (~CE1), K_7.9 (GND), L_3.15 (E), L_3.8 (GND), L_7.10 (~CE2), L_7.8 (~CE1), L_7.9 (GND)
- net P93: now also D_6.1 (S0~), D_6.18 (SL), D_7.1 (S0~), D_7.18 (SL)
- net P94: now also F_6.10 (2C0), F_6.11 (2C1), F_6.12 (2C2), F_6.13 (2C3), F_6.4 (1C2)
- net P96: now also J_3.4 (1C2), K_3.4 (1C2)
- net S1: now also E_5.6, E_6.1, F_6.14 (A), H_3.1 (S), J_3.14 (A), K_3.14 (A), L_3.1 (S)
- net S2: now also E_6.3, F_6.2 (B), H_3.15 (E), J_3.2 (B), K_3.2 (B)
- new net: B_8.9 (2S), D_6.11 (SR~)
- new net: D_6.17 (QH), D_7.11 (SR~)
- new net: B_9.1 (A), B_9.2 (B), D_7.17 (QH)
- new net: A_9.1 (A), A_9.2 (B), B_9.13 (QH)
- new net: A_9.13 (QH), B_8.7 (2B)
- new net: E_7.2, K_8.8
- new net: F_7.11, K_8.9
- new net 1.5GCLK: F_7.13
- new net 3GCLK: E_7.1
- new net BIC0: J_3.11 (2C1)
- new net BIC1: K_3.11 (2C1)
- new net BIC2: J_3.5 (1C1)
- new net BIC3: K_3.5 (1C1)
- new net BIC4: F_6.5 (1C1)
- new net BIC6: H_3.3 (1B)
- new net BIC7: H_3.13 (4B), H_3.6 (2B)
- new net BIC8: H_3.10 (3B)
- new net IP0: L_3.13 (4B), L_7.14 (D4)
- new net IP1: L_3.3 (1B), L_7.13 (D5)
- new net IP10: F_7.1, J_7.12 (D6)
- new net IP11: E_7.5, J_7.11 (D7)
- new net IP12: H_7.14 (D4)
- new net IP13: E_7.10, H_7.13 (D5)
- new net IP14: F_7.5, H_7.12 (D6)
- new net IP15: F_7.9, H_7.11 (D7)
- new net IP2: E_7.13, J_3.13 (2C3), L_7.12 (D6)
- new net IP3: K_3.13 (2C3), L_7.11 (D7)
- new net IP4: J_3.3 (1C3), K_7.14 (D4)
- new net IP5: K_3.3 (1C3), K_7.13 (D5)
- new net IP6: F_6.3 (1C3), K_7.12 (D6)
- new net IP7: E_6.2, K_7.11 (D7)
- new net IP8: D_6.19 (S1~), D_7.19 (S1~), D_8.9, J_7.14 (D4)
- new net IP9: F_7.12, J_7.13 (D5)
- new net MA0: F_5.8 (A0), H_5.8 (A0), L_3.12 (4Y)
- new net MA1: F_5.7 (A1), H_5.7 (A1), L_3.4 (1Y)
- new net MA10: F_5.19 (A10), H_3.9 (3Y), H_5.19 (A10)
- new net MA2: F_5.6 (A2), H_5.6 (A2), J_3.9 (2Y)
- new net MA3: F_5.5 (A3), H_5.5 (A3), K_3.9 (2Y)
- new net MA4: F_5.4 (A4), H_5.4 (A4), J_3.7 (1Y)
- new net MA5: F_5.3 (A5), H_5.3 (A5), K_3.7 (1Y)
- new net MA6: F_5.2 (A6), F_6.7 (1Y), H_5.2 (A6)
- new net MA7: F_5.1 (A7), H_3.12 (4Y), H_5.1 (A7)
- new net MA8: F_5.23 (A8), H_3.4 (1Y), H_5.23 (A8)
- new net MA9: F_5.22 (A9), H_3.7 (2Y), H_5.22 (A9)
- new net MDB0: D_7.16 (H~), H_5.9 (D0)
- new net MDB1: D_7.4 (G~), H_5.10 (~OE)
- new net MDB10: D_6.15 (F~), F_5.11 (D2)
- new net MDB11: D_6.5 (E~), F_5.13 (D3)
- new net MDB12: D_6.14 (D~), F_5.14 (D4)
- new net MDB13: D_6.6 (C~), F_5.15 (D5)
- new net MDB14: D_6.13 (B~), F_5.16 (D6)
- new net MDB15: D_6.7 (A~), F_5.17 (D7)
- new net MDB2: D_7.15 (F~), H_5.11 (D2)
- new net MDB3: D_7.5 (E~), H_5.13 (D3)
- new net MDB4: D_7.14 (D~), H_5.14 (D4)
- new net MDB5: D_7.6 (C~), H_5.15 (D5)
- new net MDB6: D_7.13 (B~), H_5.16 (D6)
- new net MDB7: D_7.7 (A~), H_5.17 (D7)
- new net MDB8: D_6.16 (H~), F_5.9 (D0)
- new net MDB9: D_6.4 (G~), F_5.10 (~OE)
- new net MPA0: H_7.5 (A0), J_7.5 (A0), K_7.5 (A0), L_7.5 (A0)
- new net MPA1: H_7.6 (A1), J_7.6 (A1), K_7.6 (A1), L_7.6 (A1)
- new net MPA2: H_7.7 (A2), J_7.7 (A2), K_7.7 (A2), L_7.7 (A2)
- new net MPA3: H_7.4 (A3), J_7.4 (A3), K_7.4 (A3), L_7.4 (A3)
- new net MPA4: H_7.3 (A4), J_7.3 (A4), K_7.3 (A4), L_7.3 (A4)
- new net MPA5: H_7.2 (A5), J_7.2 (A5), K_7.2 (A5), L_7.2 (A5)
- new net MPA6: H_7.1 (A6), J_7.1 (A6), K_7.1 (A6), L_7.1 (A6)
- new net MPA7: H_7.17 (A7), J_7.17 (A7), K_7.17 (A7), L_7.17 (A7)
- new net MPA8: H_7.16 (A8), J_7.16 (A8), K_7.16 (A8), L_7.16 (A8)
- new net MPA9: H_7.15 (A9), J_7.15 (A9), K_7.15 (A9), L_7.15 (A9)
- new net SERIAL_MULT: B_8.6 (2A)
- new net WP: D_8.10, E_7.12, E_7.4, E_7.9, F_7.10, F_7.2, F_7.4
- new net ~AW: H_5.21 (~WE)
- new net ~BW: F_5.21 (~WE)
- new net ~CLEAR_ACC: D_6.9 (CLR~), D_7.9 (CLR~), E_7.11
- new net ~CLR: A_9.9 (C), B_9.9 (C)
- new net ~ENA: E_5.4
- new net ~ENB: E_5.5
- new net ~GMCLK: A_9.8 (CLK), B_8.1 (CLK~), B_9.8 (CLK)
- new net ~INC_BIC: E_7.6
- new net ~LAC: D_8.8
- new net ~LDA: F_7.8
- new net ~LDB: F_7.6
- new net ~LDC: B_8.11 (CLR), E_7.8
- new net ~LW: D_6.2 (G1~), D_6.3 (G2~), D_7.2 (G1~), D_7.3 (G2~), E_7.3
- new net ~MHALT: F_7.3
- new net ~RCLK: D_6.12 (CK~), D_7.12 (CK~)
- no-connect marks 94 -> 127
Other:
- note added: "ACCUMULATOR"
- note added: "INSTRUCTION\nPROM"
- note added: "INSTRUCTION\nSTROBE GATES"
- note added: "MATRIX PROCESSOR\nADDRESS SELECTOR"
- note added: "MATRIX PROCESSOR\nRAM"

Commit message: Continued the schematic
Parts:
- added A_6, A_7, B_6, B_7: LS165A, symbol star_wars_arcade_main_pcb:LS165A
- added A_8, H_8: LS74, symbol Asteroids:LS74
- added C_10, C_9, D_9: LS161, symbol Star_Wars_Vector_PCB:LS161
- added C_6, C_7: LS384, symbol star_wars_arcade_main_pcb:LS384
- added C_8: LS08, symbol Asteroids:LS08
- added D_3, E_3, F_3: LS191_, symbol Asteroids:LS191_
- added unit 4 of D_8
- added E_8: S02, symbol Star_Wars_Vector_PCB:LS02
- added F_8: S10, symbol Asteroids:LS10
- added unit 6 of K_8
Connections:
- net +5V: now also A_6.16 (VCC), A_7.16 (VCC), A_8.14 (VCC), B_6.16 (VCC), B_7.16 (VCC), C_10.16 (VCC), C_6.16 (VCC), C_7.16 (VCC), C_8.14 (VCC), C_9.16 (VCC), D_3.16 (VCC), D_9.16 (VCC), E_3.16 (VCC), E_8.14 (VCC), F_3.16 (VCC), F_8.14 (VCC)
- net 1.5GCLK: now also D_9.13 (QB)
- net 12MHZ: now also C_10.2 (CLK), C_9.2 (CLK), D_9.2 (CLK), E_8.11, E_8.8
- net 3GCLK: now also D_9.12 (QC)
- net BIC0: now also E_3.3 (QA)
- net BIC1: now also E_3.2 (QB)
- net BIC2: now also E_3.6 (QC)
- net BIC3: now also E_3.7 (QD)
- net BIC4: now also F_3.3 (QA)
- net BIC6: now also F_3.6 (QC)
- net BIC7: now also F_3.7 (QD)
- net BIC8: now also D_3.3 (QA)
- net DB0: now also D_3.15 (A), E_3.15 (A)
- net DB1: now also E_3.1 (B)
- net DB2: now also E_3.10 (C)
- net DB3: now also E_3.9 (D)
- net DB4: now also F_3.15 (A)
- net DB5: now also F_3.1 (B)
- net DB6: now also F_3.10 (C)
- net DB7: now also F_3.9 (D)
- net GND: now also A_6.15 (~CE), A_6.8 (GND), A_7.15 (~CE), A_7.8 (GND), A_8.7 (GND), B_6.15 (~CE), B_6.8 (GND), B_7.15 (~CE), B_7.8 (GND), C_10.8 (GND), C_6.10 (K), C_6.8 (GND), C_6.9 (M), C_7.8 (GND), C_8.7 (GND), C_9.4 (B), C_9.6 (D), C_9.8 (GND), D_3.5 (D/U), D_3.8 (GND), D_9.5 (C), D_9.8 (GND), E_3.4 (G), E_3.5 (D/U), E_3.8 (GND), E_8.12, E_8.5, E_8.7 (GND), F_3.5 (D/U), F_3.8 (GND), F_8.7 (GND), H_8.12 (2D)
- net MATH_RUN: now also F_8.13, H_8.9 (2Q)
- net MDB0: now also A_7.6 (D7), B_7.6 (D7), C_7.5 (X0)
- net MDB1: now also A_7.5 (D6), B_7.5 (D6), C_7.4 (X1)
- net MDB10: now also A_6.4 (D5), B_6.4 (D5), C_6.3 (X2)
- net MDB11: now also A_6.3 (D4), B_6.3 (D4), C_6.2 (X3)
- net MDB12: now also A_6.14 (D3), B_6.14 (D3), C_6.14 (X4)
- net MDB13: now also A_6.13 (D2), B_6.13 (D2), C_6.13 (X5)
- net MDB14: now also A_6.12 (D1), B_6.12 (D1), C_6.12 (X6)
- net MDB15: now also A_6.11 (D0), A_8.12 (2D), A_8.2 (1D), B_6.11 (D0), C_6.11 (X7)
- net MDB2: now also A_7.4 (D5), B_7.4 (D5), C_7.3 (X2)
- net MDB3: now also A_7.3 (D4), B_7.3 (D4), C_7.2 (X3)
- net MDB4: now also A_7.14 (D3), B_7.14 (D3), C_7.14 (X4)
- net MDB5: now also A_7.13 (D2), B_7.13 (D2), C_7.13 (X5)
- net MDB6: now also A_7.12 (D1), B_7.12 (D1), C_7.12 (X6)
- net MDB7: now also A_7.11 (D0), B_7.11 (D0), C_7.11 (X7)
- net MDB8: now also A_6.6 (D7), B_6.6 (D7), C_6.5 (X0)
- net MDB9: now also A_6.5 (D6), B_6.5 (D6), C_6.4 (X1)
- net P92: now also C_10.1 (C), C_10.3 (A), C_10.4 (B), C_10.5 (C), C_10.6 (D), C_10.7 (EP), C_9.1 (C), C_9.3 (A), C_9.5 (C), C_9.7 (EP), D_9.1 (C), D_9.10 (ET), D_9.3 (A), D_9.4 (B), D_9.6 (D), D_9.7 (EP)
- net P93: now also B_8.13 (3S/~A), A_8.1 (~1CLR), A_8.10 (~1PRE_), A_8.13 (~1CLR), A_8.4 (~1PRE_), C_7.9 (M)
- net S1: now also H_8.13 (~1CLR)
- net SERIAL_MULT: now also C_7.6 (PROD)
- net WP: now also E_8.10, E_8.6
- net ~CLEAR_ACC: now also C_8.1
- net ~CLR: now also C_8.3
- net ~GMCLK: now also A_6.2 (CP), A_7.2 (CP), B_6.2 (CP), B_7.2 (CP), C_6.7 (CK), C_7.7 (CK), C_8.8
- net ~LAC: now also C_8.2, C_8.4
- net ~LDA: now also A_6.1 (~PL), A_7.1 (~PL), A_8.11 (2CLK)
- net ~LDB: now also A_8.3 (1CLK), B_6.1 (~PL), B_7.1 (~PL)
- net ~LDC: now also C_10.9 (LD), C_6.1 (CLR), C_7.1 (CLR), C_9.9 (LD)
- net ~MHALT: now also H_8.11 (2CLK)
- net ~MW0: now also F_8.2, H_8.10 (~1PRE_)
- net ~MW1: now also D_3.11 (LD)
- net ~MW2: now also E_3.11 (LD), F_3.11 (LD)
- net ~RCLK: now also C_8.6
- net at B_8.12 (3S): now also C_6.15 (Y), C_7.15 (Y)
- net at B_8.14 (3B): now also B_7.9 (Q7)
- net at B_8.15 (3A): now also A_7.9 (Q7)
- new net: A_6.10 (DS), A_8.9 (2Q)
- new net: A_6.9 (Q7), A_7.10 (DS)
- new net: A_8.5 (1Q), B_6.10 (DS)
- new net: B_6.9 (Q7), B_7.10 (DS)
- new net: C_6.6 (PROD), C_7.10 (K)
- new net: C_10.10 (ET), C_9.12 (QC), D_8.13, K_8.13
- new net: C_10.15 (RCO), C_9.10 (ET)
- new net: C_8.10, C_8.5, C_8.9, D_8.11
- new net: D_9.15 (RCO), E_8.3, F_8.10, F_8.11, F_8.9
- new net: D_9.9 (LD), E_8.1
- new net: E_8.9, F_8.8
- new net: E_8.2, F_8.12
- new net: D_3.4 (G), F_3.13 (RIP)
- new net: E_3.13 (RIP), F_3.4 (G)
- new net BIC5: F_3.2 (QB)
- new net ~12MHZ: D_8.12, E_8.13
- new net ~INCBIC: D_3.14 (CK), E_3.14 (CK), F_3.14 (CK)
- new net ~MACFLAG: F_8.1
- new net ~MAC_FLAG: K_8.12
- new net ~WP: E_8.4
- no-connect marks 127 -> 154
Other:
- note added: "BLOCK INDEX COUNTER"
- note added: "MATRIX PROCESSOR CLOCK"
- note added: "MULTIPLIER/ACCUMULATOR\nCLOCK"
- note added: "REGISTER A"
- note added: "REGISTER B"
- note added: "SERIAL MULTIPLIER"
- note added: "SERIAL\nSUBTRACTOR"
