File: pcb/sheet1.sch (KiCad schematic (older format))
At the start: 310 parts, among them J16 Aud_Conn, J17 Main_Connector, J18 Cat_Box_Conn, J20 J20, Q1 2N3904, Q3 Q_NPN_BCE, Q4 Q_NPN_BCE, SW3 E/F_10, SW4 D_10, Y1 12.096MHz

Commit message: Completed the schematic but not error checking
Parts:
- added unit 1 of E_5
- added unit 2 of E_6
- added F_4, H_4: LS245A, symbol star_wars_arcade_main_pcb:LS245A
- added H_6, J_6: LS191_, symbol Asteroids:LS191_
- added unit 1 of H_8
- added unit 1 of N_8
- added unit 2 of P_7
- added R_5: LS155, symbol 74xx:74LS155
Connections:
- net +5V: now also E_5.14 (VCC), F_4.20 (VCC), H_4.20 (VCC), H_6.16 (VCC), H_8.14 (VCC), J_6.16 (VCC), N_8.14 (VCC), R_5.16 (VCC)
- net 3MHZ: now also N_8.1
- net AB0: now also R_5.3 (A1)
- net DB0: now also F_4.11 (B7), H_4.11 (B7), H_6.10 (C)
- net DB1: now also F_4.12 (B6), H_4.12 (B6), H_6.9 (D)
- net DB2: now also F_4.13 (B5), H_4.13 (B5), J_6.15 (A)
- net DB3: now also F_4.14 (B4), H_4.14 (B4), J_6.1 (B)
- net DB4: now also F_4.15 (B3), H_4.15 (B3), J_6.10 (C)
- net DB5: now also F_4.16 (B2), H_4.16 (B2), J_6.9 (D)
- net DB6: now also F_4.17 (B1), H_4.17 (B1), P_7.12 (2D)
- net DB7: now also F_4.18 (B0), H_4.18 (B0), H_8.2 (1D)
- net GND: now also E_5.7 (GND), F_4.10 (GND), H_4.10 (GND), H_6.1 (B), H_6.15 (A), H_6.4 (G), H_6.5 (D/U), H_6.8 (GND), H_8.7 (GND), J_6.4 (G), J_6.5 (D/U), J_6.8 (GND), N_8.7 (GND), R_5.8 (GND)
- net MDB0: now also H_4.9 (A7)
- net MDB1: now also H_4.8 (A6)
- net MDB10: now also F_4.7 (A5)
- net MDB11: now also F_4.6 (A4)
- net MDB12: now also F_4.5 (A3)
- net MDB13: now also F_4.4 (A2)
- net MDB14: now also F_4.3 (A1)
- net MDB15: now also F_4.2 (A0)
- net MDB2: now also H_4.7 (A5)
- net MDB3: now also H_4.6 (A4)
- net MDB4: now also H_4.5 (A3)
- net MDB5: now also H_4.4 (A2)
- net MDB6: now also H_4.3 (A1)
- net MDB7: now also H_4.2 (A0)
- net MDB8: now also F_4.9 (A7)
- net MDB9: now also F_4.8 (A6)
- net MPA0: now also H_6.3 (QA)
- net MPA1: now also H_6.2 (QB)
- net MPA2: now also H_6.6 (QC)
- net MPA3: now also H_6.7 (QD)
- net MPA8: now also P_7.9 (2Q)
- net MPA9: now also H_8.5 (1Q)
- net P93: now also H_8.1 (~1CLR), H_8.4 (~1PRE_)
- net P95: now also P_7.10 (~1PRE_), P_7.13 (~1CLR), R_5.1 (Ea1)
- net R~W~B: now also F_4.1 (DIR), H_4.1 (DIR)
- net ~1.5MHZ: now also R_5.14 (Eb1), R_5.2 (Ea2)
- net ~AW: now also E_5.3
- net ~BW: now also E_6.6
- net ~ENA: now also H_4.19 (CE), R_5.5 (Q2a)
- net ~ENB: now also F_4.19 (CE), R_5.7 (Q0a)
- net ~LW: now also E_5.1, E_6.4
- net ~MBRAM: now also R_5.13 (A0)
- net ~MW0: now also H_6.11 (LD), H_8.3 (1CLK), P_7.11 (2CLK)
- net ~R~WB: now also N_8.2
- net ~WP: now also H_6.14 (CK)
- new net: E_5.2, R_5.11 (Q2b)
- new net: N_8.3, R_5.15 (Eb2)
- new net: E_6.5, R_5.9 (Q0b)
- new net MW0: J_6.11 (LD)
- new net PA4: J_6.3 (QA)
- new net PA5: J_6.2 (QB)
- new net PA6: J_6.6 (QC)
- new net PA7: J_6.7 (QD)
- new net RC: H_6.13 (RIP), J_6.14 (CK)
- no-connect marks 154 -> 163
Other:
- note added: "ADDRESS AND DATA\nSELECTOR CONTROL"
- note added: "MATRIX PROCESSOR\nADDRESS COUNTER"
- note added: "MATRIX PROCESSOR\nDATA SELECTOR"

Commit message: Fixed most schematic errors
Connections:
- net AB14 is gone; now on net A14: B/C_0.2 (B)
- net AB15 is gone; now on net A15: B/C_0.3 (C)
- net MW0 is gone; now on net ~MW0: J_6.11 (LD)
- net PA4 is gone; now on net MPA4: J_6.3 (QA)
- net PA5 is gone; now on net MPA5: J_6.2 (QB)
- net PA6 is gone; now on net MPA6: J_6.6 (QC)
- net PA7 is gone; now on net MPA7: J_6.7 (QD)
- net RWB is gone; now on net R~W~B: E_4.1 (DIR)
- net ~AB0 is gone; now on net AB0: J_2.14 (2A)
- net ~INC_BIC is gone; now on net ~INCBIC: E_7.6
- net ~MACFLAG is gone; now on net ~MAC_FLAG: F_8.1
- net 3MHZ: now also M_2.3 (1CLK), N_2.13 (QB), TP3MHZ1.1, TP3MHZ1.2
- net AB0: now also F_1.10 (A0), H/J_1.10 (A0), J/K_1.10 (A0), K/L_1.10 (A0), K_9.25 (ADDA), M_1.10 (A0)
- net AB1: now also F_1.9 (A1), H/J_1.9 (A1), J/K_1.9 (A1), K/L_1.9 (A1), M_1.9 (A1)
- net AB10: now also F_1.21 (A10), H/J_1.21 (A10), J/K_1.21 (A10), K/L_1.21 (A10), M_1.21 (A10)
- net AB11: now also F_1.23 (A11), H/J_1.23 (A11), J/K_1.23 (A11), K/L_1.23 (A11), M_1.23 (A11)
- net AB12: now also F_1.2 (A12), H/J_1.2 (A12), J/K_1.2 (A12), K/L_1.2 (A12), M_1.2 (A12)
- net AB2: now also F_1.8 (A2), H/J_1.8 (A2), J/K_1.8 (A2), K/L_1.8 (A2), M_1.8 (A2)
- net AB3: now also F_1.7 (A3), H/J_1.7 (A3), J/K_1.7 (A3), K/L_1.7 (A3), M_1.7 (A3)
- net AB4: now also F_1.6 (A4), H/J_1.6 (A4), J/K_1.6 (A4), K/L_1.6 (A4), M_1.6 (A4)
- net AB5: now also F_1.5 (A5), H/J_1.5 (A5), J/K_1.5 (A5), K/L_1.5 (A5), M_1.5 (A5)
- net AB6: now also F_1.4 (A6), H/J_1.4 (A6), J/K_1.4 (A6), K/L_1.4 (A6), M_1.4 (A6)
- net AB7: now also F_1.3 (A7), H/J_1.3 (A7), J/K_1.3 (A7), K/L_1.3 (A7), M_1.3 (A7)
- net AB8: now also F_1.25 (A8), H/J_1.25 (A8), J/K_1.25 (A8), K/L_1.25 (A8), M_1.25 (A8)
- net AB9: now also F_1.24 (A9), H/J_1.24 (A9), J/K_1.24 (A9), K/L_1.24 (A9), M_1.24 (A9)
- net IP12: now also E_7.13
- net IP2: no longer E_7.13
- net ~PITCH: now also R79.2
- net ~THRUST: no longer R79.2
- removed net AB: F_1.10 (A0), F_1.2 (A12), F_1.21 (A10), F_1.23 (A11), F_1.24 (A9), F_1.25 (A8), F_1.3 (A7), F_1.4 (A6), F_1.5 (A5), F_1.6 (A4), F_1.7 (A3), F_1.8 (A2), F_1.9 (A1), H/J_1.10 (A0), H/J_1.2 (A12), H/J_1.21 (A10), H/J_1.23 (A11), H/J_1.24 (A9), H/J_1.25 (A8), H/J_1.3 (A7), H/J_1.4 (A6), H/J_1.5 (A5), H/J_1.6 (A4), H/J_1.7 (A3), H/J_1.8 (A2), H/J_1.9 (A1), J/K_1.10 (A0), J/K_1.2 (A12), J/K_1.21 (A10), J/K_1.23 (A11), J/K_1.24 (A9), J/K_1.25 (A8), J/K_1.3 (A7), J/K_1.4 (A6), J/K_1.5 (A5), J/K_1.6 (A4), J/K_1.7 (A3), J/K_1.8 (A2), J/K_1.9 (A1), K/L_1.10 (A0), K/L_1.2 (A12), K/L_1.21 (A10), K/L_1.23 (A11), K/L_1.24 (A9), K/L_1.25 (A8), K/L_1.3 (A7), K/L_1.4 (A6), K/L_1.5 (A5), K/L_1.6 (A4), K/L_1.7 (A3), K/L_1.8 (A2), K/L_1.9 (A1), M_1.10 (A0), M_1.2 (A12), M_1.21 (A10), M_1.23 (A11), M_1.24 (A9), M_1.25 (A8), M_1.3 (A7), M_1.4 (A6), M_1.5 (A5), M_1.6 (A4), M_1.7 (A3), M_1.8 (A2), M_1.9 (A1)
Changed lines of the file:
@@
 	11925 3400 12775 3400
 Wire Wire Line
-	13200 3550 12125 3550
+	13200 3550 13000 3550
 Wire Wire Line
 	11825 3550 11825 3125
@@
 	20350 6075 20450 6075
 Text GLabel 21025 6475 0    50   Input ~ 0
-RWB
+R~W~B
 $Comp
 L Asteroids:LS08 K_6
@@
 	26300 1625 25825 1625
 Text GLabel 25825 1725 0    50   Input ~ 0
-AB
+AB12
 Text GLabel 25825 1825 0    50   Input ~ 0
-AB
+AB11
 Text GLabel 25825 1925 0    50   Input ~ 0
-AB
+AB10
 Text GLabel 25825 2025 0    50   Input ~ 0
-AB
+AB9
 Text GLabel 25825 2125 0    50   Input ~ 0
-AB
+AB8
 Text GLabel 25825 2225 0    50   Input ~ 0
-AB
+AB7
 Text GLabel 25825 2325 0    50   Input ~ 0
-AB
+AB6
 Text GLabel 25825 2425 0    50   Input ~ 0
-AB
+AB5
 Text GLabel 25825 2525 0    50   Input ~ 0
-AB
+AB4
 Text GLabel 25825 2625 0    50   Input ~ 0
-AB
+AB3
 Text GLabel 25825 2725 0    50   Input ~ 0
-AB
+AB2
 Text GLabel 25825 2825 0    50   Input ~ 0
-AB
+AB1
 Text GLabel 25825 2925 0    50   Input ~ 0
-AB
+AB0
 Wire Wire Line
 	26300 1725 25825 1725
@@
 P92
 Text GLabel 41300 1950 0    50   Input ~ 0
-AB15
+A15
 Text GLabel 41300 2050 0    50   Input ~ 0
-AB14
+A14
 Text GLabel 41300 2150 0    50   Input ~ 0
 AB13
@@
 AB1
 Text GLabel 28300 8625 0    50   Input ~ 0
-~AB0
+AB0
 Text Notes 26075 6375 0    200  ~ 0
 MATH ADDRESS DECODERS
@@
 Connection ~ 21950 9900
 Text GLabel 21575 9900 0    50   Input ~ 0
-~THRUST
+~PITCH
 Wire Wire Line
 	21950 10350 21950 10400
@@
 Connection ~ 24525 11250
 Wire Wire Line
-	24550 11050 23425 11050
+	24575 11050 23425 11050
 Wire Wire Line
 	23425 11050 23425 11650
@@
 ~MHALT
 Text GLabel 36700 29275 2    50   Input ~ 0
-~INC_BIC
+~INCBIC
 Text GLabel 36700 29900 2    50   Input ~ 0
 ~CLEAR_ACC
@@
 IP11
 Text GLabel 35500 29800 0    50   Input ~ 0
-IP2
+IP12
 Text GLabel 35500 30425 0    50   Input ~ 0
 IP13
@@
 Connection ~ 5825 19275
 Text GLabel 6050 18300 0    50   Input ~ 0
-~MACFLAG
+~MAC_FLAG
 $Comp
 L power:GND #PWR0475
@@
 DB2
 Text GLabel 19000 18900 1    50   Input ~ 0
-MW0
+~MW0
 Text GLabel 19400 20300 3    50   Input ~ 0
-PA7
+MPA7
 Text GLabel 19300 20300 3    50   Input ~ 0
-PA6
+MPA6
 Text GLabel 19200 20300 3    50   Input ~ 0
-PA5
+MPA5
 Text GLabel 19100 20300 3    50   Input ~ 0
-PA4
+MPA4
 Text GLabel 19000 20300 3    50   Input ~ 0
 RC
@@
 AB0
 $Comp
-L power:GND #PWR?
+L power:GND #PWR0498
 U 1 1 A870833E
 P 24050 20050
-F 0 "#PWR?" H 24050 19800 50  0001 C CNN
+F 0 "#PWR0498" H 24050 19800 50  0001 C CNN
 F 1 "GND" H 24200 20050 50  0000 C CNN
 F 2 "" H 24050 20050 50  0001 C CNN
@@
 $EndComp
 $Comp
-L power:+5V #PWR?
+L power:+5V #PWR0499
 U 1 1 A8709313
 P 24050 18650
-F 0 "#PWR?" H 24050 18500 50  0001 C CNN
+F 0 "#PWR0499" H 24050 18500 50  0001 C CNN
 F 1 "+5V" H 24175 18650 50  0000 C CNN
 F 2 "" H 24050 18650 50  0001 C CNN
@@
 3MHZ
 $Comp
-L power:+5V #PWR?
+L power:+5V #PWR0500
 U 1 1 AA2B8A6D
 P 22475 19450
-F 0 "#PWR?" H 22475 19300 50  0001 C CNN
+F 0 "#PWR0500" H 22475 19300 50  0001 C CNN
 F 1 "+5V" H 22490 19623 50  0000 C CNN
 F 2 "" H 22475 19450 50  0001 C CNN
@@
 $EndComp
 $Comp
-L power:GND #PWR?
+L power:GND #PWR0501
 U 1 1 AA2B9ADD
 P 22475 19850
-F 0 "#PWR?" H 22475 19600 50  0001 C CNN
+F 0 "#PWR0501" H 22475 19600 50  0001 C CNN
 F 1 "GND" H 22480 19677 50  0000 C CNN
 F 2 "" H 22475 19850 50  0001 C CNN
@@
 $EndComp
 $Comp
-L power:GND #PWR?
+L power:GND #PWR0502
 U 1 1 AAEAA96B
 P 24050 21300
-F 0 "#PWR?" H 24050 21050 50  0001 C CNN
+F 0 "#PWR0502" H 24050 21050 50  0001 C CNN
 F 1 "GND" H 24055 21127 50  0000 C CNN
 F 2 "" H 24050 21300 50  0001 C CNN
@@
 $EndComp
 $Comp
-L power:+5V #PWR?
+L power:+5V #PWR0503
 U 1 1 AAEAAFBB
 P 24050 21700
-F 0 "#PWR?" H 24050 21550 50  0001 C CNN
+F 0 "#PWR0503" H 24050 21550 50  0001 C CNN
 F 1 "+5V" H 24065 21873 50  0000 C CNN
 F 2 "" H 24050 21700 50  0001 C CNN
@@
 Wire Notes Line
 	25150 17850 21600 17850
+Text GLabel 13000 3675 3    50   Input ~ 0
+3MHZ
+Wire Wire Line
+	13000 3675 13000 3550
+Connection ~ 13000 3550
+Wire Wire Line
+	13000 3550 12125 3550
+$Comp
+L power:PWR_FLAG #FLG0101
+U 1 1 AEB8AB6F
+P 4500 6875
+F 0 "#FLG0101" H 4500 6950 50  0001 C CNN
+F 1 "PWR_FLAG" H 4500 7048 50  0000 C CNN
+F 2 "" H 4500 6875 50  0001 C CNN
+F 3 "~" H 4500 6875 50  0001 C CNN
+	1    4500 6875
+	1    0    0    -1
+$EndComp
+$Comp
+L power:+10V #PWR0504
+U 1 1 AEB8CC9C
+P 4500 6875
+F 0 "#PWR0504" H 4500 6725 50  0001 C CNN
+F 1 "+10V" V 4515 7003 50  0000 L CNN
+F 2 "" H 4500 6875 50  0001 C CNN
+F 3 "" H 4500 6875 50  0001 C CNN
+	1    4500 6875
+	-1   0    0    1
+$EndComp
+$Comp
+L power:+12V #PWR0505
+U 1 1 AEF97AD0
+P 4925 6875
+F 0 "#PWR0505" H 4925 6725 50  0001 C CNN
+F 1 "+12V" V 4940 7003 50  0000 L CNN
+F 2 "" H 4925 6875 50  0001 C CNN
+F 3 "" H 4925 6875 50  0001 C CNN
+	1    4925 6875
+	-1   0    0    1
+$EndComp
+$Comp
+L power:PWR_FLAG #FLG0102
+U 1 1 AF397A6C
+P 4925 6875
+F 0 "#FLG0102" H 4925 6950 50  0001 C CNN
+F 1 "PWR_FLAG" H 4925 7048 50  0000 C CNN
+F 2 "" H 4925 6875 50  0001 C CNN
+F 3 "~" H 4925 6875 50  0001 C CNN
+	1    4925 6875
+	1    0    0    -1
+$EndComp
+$Comp
+L power:-5V #PWR0506
+U 1 1 AF7B04BF
+P 5350 6875
+F 0 "#PWR0506" H 5350 6975 50  0001 C CNN
+F 1 "-5V" V 5365 7003 50  0000 L CNN
+F 2 "" H 5350 6875 50  0001 C CNN
+F 3 "" H 5350 6875 50  0001 C CNN
+	1    5350 6875
+	-1   0    0    1
+$EndComp
+$Comp
+L power:PWR_FLAG #FLG0103
+U 1 1 AFBAFA29
+P 5350 6875
+F 0 "#FLG0103" H 5350 6950 50  0001 C CNN
+F 1 "PWR_FLAG" H 5350 7048 50  0000 C CNN
+F 2 "" H 5350 6875 50  0001 C CNN
+F 3 "~" H 5350 6875 50  0001 C CNN
+	1    5350 6875
+	1    0    0    -1
+$EndComp
 $EndSCHEMATC

Commit message: Fixed all errors on the schematic
Connections:
- net BIC5: now also H_3.13 (4B)
- net BIC7: no longer H_3.13 (4B)
- net 46KHZ: no longer names the net of P_2.1 (1CK), P_2.8 (2QD)
- net P: no longer names the net of M_7.9 (CLR~)
- no-connect marks 163 -> 164
Other:
- note added: "No Connection on PCB"
Changed lines of the file:
@@
 Wire Wire Line
 	13450 4450 13300 4450
-Text GLabel 13600 4450 2    50   Input ~ 0
-46KHZ
-Wire Wire Line
-	13600 4450 13450 4450
-Connection ~ 13450 4450
 Wire Wire Line
 	13300 4950 13375 4950
@@
 Wire Wire Line
 	35725 17450 36125 17450
-Text GLabel 37425 18725 0    50   Input ~ 0
-P
 Text GLabel 37225 18825 0    50   Input ~ 0
 ~REN
@@
 BIC6
 Text GLabel 25150 26425 0    50   Input ~ 0
-BIC7
+BIC5
 $Comp
 L power:GND #PWR0381
@@
 	1    0    0    -1
 $EndComp
+Text Notes 35975 18775 0    50   ~ 0
+No Connection on PCB
+NoConn ~ 37425 18725
+Wire Notes Line
+	36875 18725 37400 18725
 $EndSCHEMATC

Commit message: Began the PCB layout
Parts:
- added SPARE1: SpareB, Star_Wars_Vector_PCB:DIP16, symbol Star_Wars_Vector_PCB:SpareB
- B/C_0, P_4, P_5, P_6, P_8, R_3, R_5, R_8: footprint (none) -> Star_Wars_Vector_PCB:DIP16
- B_1, C_1, D/E0: footprint (none) -> Star_Wars_Vector_PCB:DIP20
- E_1: footprint (none) -> Star_Wars_Vector_PCB:DIP18
- F_1, H/J_1, J/K_1, K/L_1, M_1: footprint (none) -> Star_Wars_Main_PCB:DIP28
- J18: footprint (none) -> Asteroids:J21
- J20: footprint (none) -> Asteroids:Edge_Connector
- N_1, P_2, P_3, P_7, R_10, R_2, R_6: footprint (none) -> Star_Wars_Vector_PCB:DIP14
Connections:
- net +5V: now also SPARE1.16 (VCC)
- net GND: now also SPARE1.8 (GND)
- no-connect marks 164 -> 178
Changed lines of the file:
@@
 F 0 "J20" H 44650 27983 50  0000 C CNN
 F 1 "J20" H 44600 28000 50  0001 C CNN
-F 2 "" H 44550 27450 50  0001 C CNN
+F 2 "Asteroids:Edge_Connector" H 44550 27450 50  0001 C CNN
 F 3 "" H 44550 27450 50  0001 C CNN
 	1    44650 26800
@@
 F 0 "J18" H 44575 31297 60  0000 C CNN
 F 1 "Cat_Box_Conn" H 44575 31191 60  0000 C CNN
-F 2 "" H 44825 29650 60  0001 C CNN
+F 2 "Asteroids:J21" H 44825 29650 60  0001 C CNN
 F 3 "" H 44825 29650 60  0001 C CNN
 	1    44600 29850
@@
 F 0 "N_1" H 9725 2775 50  0000 C CNN
 F 1 "S04" H 9650 2650 50  0000 C CNN
-F 2 "" H 9675 2650 50  0001 C CNN
+F 2 "Star_Wars_Vector_PCB:DIP14" H 9675 2650 50  0001 C CNN
 F 3 "" H 9675 2650 50  0001 C CNN
 	5    9675 2650
@@
 F 0 "N_1" H 9725 3250 50  0000 C CNN
 F 1 "S04" H 9625 3125 50  0000 C CNN
-F 2 "" H 9675 3125 50  0001 C CNN
+F 2 "Star_Wars_Vector_PCB:DIP14" H 9675 3125 50  0001 C CNN
 F 3 "" H 9675 3125 50  0001 C CNN
 	6    9675 3125
@@
 F 0 "N_1" H 8750 3250 50  0000 C CNN
 F 1 "S04" H 8650 3125 50  0000 C CNN
-F 2 "" H 8675 3125 50  0001 C CNN
+F 2 "Star_Wars_Vector_PCB:DIP14" H 8675 3125 50  0001 C CNN
 F 3 "" H 8675 3125 50  0001 C CNN
 	1    8675 3125
@@
 F 0 "P_2" H 12750 4875 50  0000 C CNN
 F 1 "LS393" H 12750 4800 50  0000 C CNN
-F 2 "" H 12750 4850 50  0001 C CNN
+F 2 "Star_Wars_Vector_PCB:DIP14" H 12750 4850 50  0001 C CNN
 F 3 "" H 12750 4850 50  0001 C CNN
 	1    12750 4850
@@
 F 0 "P_3" H 13400 1175 50  0000 C CNN
 F 1 "LS04" H 13400 1025 50  0000 C CNN
-F 2 "" H 13225 1100 50  0001 C CNN
+F 2 "Star_Wars_Vector_PCB:DIP14" H 13225 1100 50  0001 C CNN
 F 3 "" H 13225 1100 50  0001 C CNN
 	1    13225 1100
@@
 F 0 "R_8" H 36625 10900 50  0000 L CNN
 F 1 "LS191_" H 36575 10800 50  0000 L CNN
-F 2 "" V 36700 10850 50  0001 C CNN
+F 2 "Star_Wars_Vector_PCB:DIP16" V 36700 10850 50  0001 C CNN
 F 3 "" V 36700 10850 50  0001 C CNN
 	1    36700 10850
@@
 F 0 "P_8" H 36625 12850 50  0000 L CNN
 F 1 "LS109" H 36575 12775 50  0000 L CNN
-F 2 "" H 36700 12850 50  0001 C CNN
+F 2 "Star_Wars_Vector_PCB:DIP16" H 36700 12850 50  0001 C CNN
 F 3 "" H 36700 12850 50  0001 C CNN
 	1    36700 12850
@@
 F 0 "P_8" H 36700 14925 50  0000 C CNN
 F 1 "LS109" H 36700 14825 50  0000 C CNN
-F 2 "" H 36700 14900 50  0001 C CNN
+F 2 "Star_Wars_Vector_PCB:DIP16" H 36700 14900 50  0001 C CNN
 F 3 "" H 36700 14900 50  0001 C CNN
 	2    36700 14900
@@
 F 0 "P_7" H 44075 15175 50  0000 L CNN
 F 1 "LS74" H 44075 15100 50  0000 L CNN
-F 2 "" H 44175 14875 300 0001 C CNN
+F 2 "Star_Wars_Vector_PCB:DIP14" H 44175 14875 300 0001 C CNN
 F 3 "" H 44175 14875 300 0001 C CNN
 	1    44150 15125
@@
 F 0 "P_3" H 44200 17575 50  0000 C CNN
 F 1 "LS04" H 44200 17375 50  0000 C CNN
-F 2 "" H 44100 17475 50  0001 C CNN
+F 2 "Star_Wars_Vector_PCB:DIP14" H 44100 17475 50  0001 C CNN
 F 3 "" H 44100 17475 50  0001 C CNN
 	5    44100 17475
@@
 F 0 "P_5" H 27350 11150 50  0000 C CNN
 F 1 "LS175A" H 27350 11050 50  0000 C CNN
-F 2 "" H 27250 11100 50  0001 C CNN
+F 2 "Star_Wars_Vector_PCB:DIP16" H 27250 11100 50  0001 C CNN
 F 3 "" H 27250 11100 50  0001 C CNN
 	1    27350 11100
@@
 F 0 "P_4" H 27350 13000 50  0000 C CNN
 F 1 "LS175B" H 27325 12925 50  0000 C CNN
-F 2 "" H 27350 12925 50  0001 C CNN
+F 2 "Star_Wars_Vector_PCB:DIP16" H 27350 12925 50  0001 C CNN
 F 3 "" H 27350 12925 50  0001 C CNN
 	1    27350 12925
@@
 F 0 "P_6" H 27325 14750 50  0000 C CNN
 F 1 "LS175C" H 27350 14675 50  0000 C CNN
-F 2 "" H 27350 14725 50  0001 C CNN
+F 2 "Star_Wars_Vector_PCB:DIP16" H 27350 14725 50  0001 C CNN
 F 3 "" H 27350 14725 50  0001 C CNN
 	1    27350 14725
@@
 F 0 "R_6" H 31900 11050 50  0000 C CNN
 F 1 "LS74" H 31900 10975 50  0000 C CNN
-F 2 "" H 31925 10775 300 0001 C CNN
+F 2 "Star_Wars_Vector_PCB:DIP14" H 31925 10775 300 0001 C CNN
 F 3 "" H 31925 10775 300 0001 C CNN
 	2    31900 11025
@@
 F 0 "B_1" H 21050 2000 50  0000 C CNN
 F 1 "LS244B" H 21050 2075 50  0000 C CNN
-F 2 "" H 21050 2425 50  0001 C CNN
+F 2 "Star_Wars_Vector_PCB:DIP20" H 21050 2425 50  0001 C CNN
 F 3 "" H 21050 2425 50  0001 C CNN
 	1    21050 2425
@@
 F 0 "C_1" H 22425 4475 50  0000 C CNN
 F 1 "LS244C" H 22425 4575 50  0000 C CNN
-F 2 "" H 22425 4300 50  0001 C CNN
+F 2 "Star_Wars_Vector_PCB:DIP20" H 22425 4300 50  0001 C CNN
 F 3 "" H 22425 4300 50  0001 C CNN
 	1    22425 4300
@@
 F 0 "P_3" H 21075 7525 50  0000 C CNN
 F 1 "LS04" H 21075 7325 50  0000 C CNN
-F 2 "" H 20950 7425 50  0001 C CNN
+F 2 "Star_Wars_Vector_PCB:DIP14" H 20950 7425 50  0001 C CNN
 F 3 "" H 20950 7425 50  0001 C CNN
 	4    20950 7425
@@
 F 0 "N_1" H 22300 7525 50  0000 C CNN
 F 1 "S04" H 22275 7325 50  0000 C CNN
-F 2 "" H 22200 7425 50  0001 C CNN
+F 2 "Star_Wars_Vector_PCB:DIP14" H 22200 7425 50  0001 C CNN
 F 3 "" H 22200 7425 50  0001 C CNN
 	2    22200 7425
@@
 F 0 "D/E0" H 24150 2425 50  0000 C CNN
 F 1 "LS245A" H 24150 2325 50  0000 C CNN
-F 2 "" H 24150 2150 50  0001 C CNN
+F 2 "Star_Wars_Vector_PCB:DIP20" H 24150 2150 50  0001 C CNN
 F 3 "" H 24150 2150 50  0001 C CNN
 	1    24150 2150
@@
 F 0 "R_10" H 8900 6200 50  0000 C CNN
 F 1 "LS14" H 8900 6000 50  0000 C CNN
-F 2 "" H 8875 6100 50  0001 C CNN
+F 2 "Star_Wars_Vector_PCB:DIP14" H 8875 6100 50  0001 C CNN
 F 3 "" H 8875 6100 50  0001 C CNN
 	5    8775 6100
@@
 F 0 "R_2" H 12275 7425 50  0000 C CNN
 F 1 "LS393A" H 12275 7350 50  0000 C CNN
-F 2 "" H 12275 7375 50  0001 C CNN
+F 2 "Star_Wars_Vector_PCB:DIP14" H 12275 7375 50  0001 C CNN
 F 3 "" H 12275 7375 50  0001 C CNN
 	1    12275 7375
@@
 F 0 "R_10" H 10900 6375 50  0000 C CNN
 F 1 "LS14" H 10875 6575 50  0000 C CNN
-F 2 "" H 10850 6475 50  0001 C CNN
+F 2 "Star_Wars_Vector_PCB:DIP14" H 10850 6475 50  0001 C CNN
 F 3 "" H 10850 6475 50  0001 C CNN
 	4    10750 6475
@@
 F 0 "R_6" H 15775 7150 50  0000 L CNN
 F 1 "LS74" H 15775 7075 50  0000 L CNN
-F 2 "" H 15900 6850 300 0001 C CNN
+F 2 "Star_Wars_Vector_PCB:DIP14" H 15900 6850 300 0001 C CNN
 F 3 "" H 15900 6850 300 0001 C CNN
 	1    15875 7100
@@
 F 0 "R_3" H 10625 9325 60  0000 L CNN
 F 1 "LS161" H 10600 9250 60  0000 L CNN
-F 2 "" H 10600 9700 60  0001 C CNN
+F 2 "Star_Wars_Vector_PCB:DIP16" H 10600 9700 60  0001 C CNN
 F 3 "" H 10600 9700 60  0001 C CNN
 	1    10700 9275
@@
 F 0 "P_3" H 12225 9350 50  0000 C CNN
 F 1 "LS04" H 12225 9200 50  0000 C CNN
-F 2 "" H 12075 9275 50  0001 C CNN
+F 2 "Star_Wars_Vector_PCB:DIP14" H 12075 9275 50  0001 C CNN
 F 3 "" H 12075 9275 50  0001 C CNN
 	2    12075 9275
@@
 F 0 "F_1" H 26750 2575 50  0000 R CNN
 F 1 "27128" H 26825 2500 50  0000 R CNN
-F 2 "" H 26700 2775 50  0001 C CNN
+F 2 "Star_Wars_Main_PCB:DIP28" H 26700 2775 50  0001 C CNN
 F 3 "" H 26700 2775 50  0001 C CNN
 	1    26700 2525
@@
 F 0 "H/J_1" H 27625 2575 50  0000 R CNN
 F 1 "2764" H 27600 2500 50  0000 R CNN
-F 2 "" H 27500 2525 50  0001 C CNN
+F 2 "Star_Wars_Main_PCB:DIP28" H 27500 2525 50  0001 C CNN
 F 3 "" H 27500 2525 50  0001 C CNN
 	1    27500 2525
@@
 F 0 "J/K_1" H 28400 2575 50  0000 R CNN
 F 1 "2764" H 28400 2500 50  0000 R CNN
-F 2 "" H 28300 2525 50  0001 C CNN
+F 2 "Star_Wars_Main_PCB:DIP28" H 28300 2525 50  0001 C CNN
 F 3 "" H 28300 2525 50  0001 C CNN
 	1    28300 2525
@@
 F 0 "K/L_1" H 29225 2575 50  0000 R CNN
 F 1 "2764" H 29200 2500 50  0000 R CNN
-F 2 "" H 29100 2525 50  0001 C CNN
+F 2 "Star_Wars_Main_PCB:DIP28" H 29100 2525 50  0001 C CNN
 F 3 "" H 29100 2525 50  0001 C CNN
 	1    29100 2525
@@
 F 0 "M_1" H 29950 2575 50  0000 R CNN
 F 1 "2764" H 30000 2500 50  0000 R CNN
-F 2 "" H 29900 2525 50  0001 C CNN
+F 2 "Star_Wars_Main_PCB:DIP28" H 29900 2525 50  0001 C CNN
 F 3 "" H 29900 2525 50  0001 C CNN
 	1    29900 2525
@@
 F 0 "E_1" H 34900 2250 50  0000 C CNN
 F 1 "x2212" H 34925 2175 50  0000 C CNN
-F 2 "" H 34900 2225 50  0001 C CNN
+F 2 "Star_Wars_Vector_PCB:DIP18" H 34900 2225 50  0001 C CNN
 F 3 "" H 34900 2225 50  0001 C CNN
 	1    34900 2225
@@
 F 0 "B/C_0" H 41800 2250 50  0000 C CNN
 F 1 "LS138" H 41800 2175 50  0000 C CNN
-F 2 "" H 41800 2000 50  0001 C CNN
+F 2 "Star_Wars_Vector_PCB:DIP16" H 41800 2000 50  0001 C CNN
 F 3 "" H 41800 2000 50  0001 C CNN
 	1    41800 2000
@@
 F 0 "P_3" H 43250 5575 50  0000 C CNN
 F 1 "LS04" H 43275 5400 50  0000 C CNN
-F 2 "" H 43125 5475 50  0001 C CNN
+F 2 "Star_Wars_Vector_PCB:DIP14" H 43125 5475 50  0001 C CNN
 F 3 "" H 43125 5475 50  0001 C CNN
 	6    43125 5475
@@
 F 0 "P_7" H 19250 17950 50  0000 C CNN
 F 1 "LS74" H 19250 17875 50  0000 C CNN
-F 2 "" H 19275 17675 300 0001 C CNN
+F 2 "Star_Wars_Vector_PCB:DIP14" H 19275 17675 300 0001 C CNN
 F 3 "" H 19275 17675 300 0001 C CNN
 	2    19250 17925
@@
 F 0 "R_5" H 24050 19425 50  0000 C CNN
 F 1 "LS155" H 24075 19350 50  0000 C CNN
-F 2 "" H 24050 19350 50  0001 C CNN
+F 2 "Star_Wars_Vector_PCB:DIP16" H 24050 19350 50  0001 C CNN
 F 3 "http://www.ti.com/lit/gpn/sn74LS155" H 24050 19350 50  0001 C CNN
 	1    24050 19350
@@
 Wire Notes Line
 	36875 18725 37400 18725
+$Comp
+L Star_Wars_Vector_PCB:SpareB SPARE1
+U 1 1 616113CB
+P 40425 30875
+F 0 "SPARE1" H 40425 30975 50  0000 C CNN
+F 1 "SpareB" H 40425 30775 50  0000 C CNN
+F 2 "Star_Wars_Vector_PCB:DIP16" H 40425 30875 50  0001 C CNN
+F 3 "" H 40425 30875 50  0001 C CNN
+	1    40425 30875
+	1    0    0    -1
+$EndComp
+$Comp
+L power:+5V #PWR0507
+U 1 1 6161CEC9
+P 40425 30325
+F 0 "#PWR0507" H 40425 30175 50  0001 C CNN
+F 1 "+5V" H 40440 30498 50  0000 C CNN
+F 2 "" H 40425 30325 50  0001 C CNN
+F 3 "" H 40425 30325 50  0001 C CNN
+	1    40425 30325
+	1    0    0    -1
+$EndComp
+$Comp
+L power:GND #PWR0508
+U 1 1 616223BB
+P 40425 31425
+F 0 "#PWR0508" H 40425 31175 50  0001 C CNN
+F 1 "GND" H 40430 31252 50  0000 C CNN
+F 2 "" H 40425 31425 50  0001 C CNN
+F 3 "" H 40425 31425 50  0001 C CNN
+	1    40425 31425
+	1    0    0    -1
+$EndComp
+NoConn ~ 39725 30575
+NoConn ~ 39725 30675
+NoConn ~ 39725 30775
+NoConn ~ 39725 30875
+NoConn ~ 39725 30975
+NoConn ~ 39725 31075
+NoConn ~ 39725 31175
+NoConn ~ 41125 31175
+NoConn ~ 41125 31075
+NoConn ~ 41125 30975
+NoConn ~ 41125 30875
+NoConn ~ 41125 30775
+NoConn ~ 41125 30675
+NoConn ~ 41125 30575
 $EndSCHEMATC
