File: pcb/star_wars_arcade_main_pcb.kicad_pcb (KiCad board)
At the start: 2 copper layers, 292.1 x 525.8 mm, 32 parts, among them J17 Main_Connector, J18 Cat_Box_Conn, J20 J20

Commit message: Placed all the ICs
Parts:
- added A_6: LS165A, Star_Wars_Vector_PCB:DIP16, F.Cu at (302.9, 281.3)
- added A_7: LS165A, Star_Wars_Vector_PCB:DIP16, F.Cu at (302.9, 244.5)
- added A_8: LS74, Star_Wars_Vector_PCB:DIP14, F.Cu at (302.9, 205.1)
- added A_9: LS164A, Star_Wars_Vector_PCB:DIP14, F.Cu at (302.9, 160.0)
- added B_5: LS86, Star_Wars_Vector_PCB:DIP14, F.Cu at (283.2, 319.4)
- added B_6: LS165A, Star_Wars_Vector_PCB:DIP16, F.Cu at (283.2, 281.3)
- added B_7: LS165A, Star_Wars_Vector_PCB:DIP16, F.Cu at (283.2, 244.5)
- added B_8: LS385, Star_Wars_Vector_PCB:DIP20, F.Cu at (283.2, 205.1)
- added B_9: LS164A, Star_Wars_Vector_PCB:DIP14, F.Cu at (283.2, 160.0)
- added C_10: LS161, Star_Wars_Vector_PCB:DIP16, F.Cu at (262.3, 112.4)
- added C_2: 68B09E, Star_Wars_Vector_PCB:DDIP40, F.Cu at (256.5, 436.9)
- added C_5: LS164A, Star_Wars_Vector_PCB:DIP14, F.Cu at (262.3, 319.4)
- added C_6: LS384, Star_Wars_Vector_PCB:DIP16, F.Cu at (262.3, 281.3)
- added C_7: LS384, Star_Wars_Vector_PCB:DIP16, F.Cu at (262.3, 244.5)
- added C_8: LS08, Star_Wars_Vector_PCB:DIP14, F.Cu at (262.3, 205.1)
- added C_9: LS161, Star_Wars_Vector_PCB:DIP16, F.Cu at (262.3, 160.0)
- added D_3: LS191_, Star_Wars_Vector_PCB:DIP16, F.Cu at (245.7, 397.5)
- added D_4: LS299, Star_Wars_Vector_PCB:DIP20, F.Cu at (245.7, 359.4)
- added D_5: LS164A, Star_Wars_Vector_PCB:DIP14, F.Cu at (241.9, 319.4)
- added D_6: LS299, Star_Wars_Vector_PCB:DIP20, F.Cu at (241.9, 281.3)
- added D_7: LS299, Star_Wars_Vector_PCB:DIP20, F.Cu at (241.3, 244.5)
- added D_8: LS00, Star_Wars_Vector_PCB:DIP14, F.Cu at (241.3, 205.1)
- added D_9: LS161, Star_Wars_Vector_PCB:DIP16, F.Cu at (241.3, 160.0)
- added E/F_2: LS244D, Star_Wars_Vector_PCB:DIP20, F.Cu at (212.1, 435.6)
- added E_3: LS191_, Star_Wars_Vector_PCB:DIP16, F.Cu at (221.6, 397.5)
- added E_4: LS245A, Star_Wars_Vector_PCB:DIP20, F.Cu at (221.6, 359.4)
- added E_5: LS08, Star_Wars_Vector_PCB:DIP14, F.Cu at (221.6, 319.4)
- added E_6: LS08, Star_Wars_Vector_PCB:DIP14, F.Cu at (221.6, 281.3)
- added E_7: LS00, Star_Wars_Vector_PCB:DIP14, F.Cu at (221.6, 244.5)
- added E_8: S02, Star_Wars_Vector_PCB:DIP14, F.Cu at (221.6, 205.1)
- added E_9: LS244, Star_Wars_Vector_PCB:DIP20, F.Cu at (221.6, 160.0)
- added F/H_2: 137211, Star_Wars_Vector_PCB:DDIP24, F.Cu at (189.9, 435.6)
- added F_3: LS191_, Star_Wars_Vector_PCB:DIP16, F.Cu at (200.7, 397.5)
- added F_4: LS245A, Star_Wars_Vector_PCB:DIP20, F.Cu at (200.7, 359.4)
- added F_5: RAM, Star_Wars_Vector_PCB:DDIP24, F.Cu at (204.5, 316.9)
- added F_6: LS153A, Star_Wars_Vector_PCB:DIP16, F.Cu at (200.7, 281.3)
- added F_7: LS00, Star_Wars_Vector_PCB:DIP14, F.Cu at (200.7, 244.5)
- added F_8: S10, Star_Wars_Vector_PCB:DIP14, F.Cu at (200.7, 205.1)
- added F_9: LS244, Star_Wars_Vector_PCB:DIP20, F.Cu at (200.7, 160.0)
- added H_3: LS157A, Star_Wars_Vector_PCB:DIP16, F.Cu at (180.3, 397.5)
- added H_4: LS245A, Star_Wars_Vector_PCB:DIP20, F.Cu at (180.3, 359.4)
- added H_5: RAM, Star_Wars_Vector_PCB:DDIP24, F.Cu at (177.8, 316.9)
- added H_6: LS191_, Star_Wars_Vector_PCB:DIP16, F.Cu at (180.3, 281.3)
- added H_7: PROM, Star_Wars_Vector_PCB:DIP18, F.Cu at (180.3, 244.5)
- added H_8: LS74, Star_Wars_Vector_PCB:DIP14, F.Cu at (180.3, 205.1)
- added H_9: LS244E, Star_Wars_Vector_PCB:DIP20, F.Cu at (175.9, 160.0)
- added J_2: LS139, Star_Wars_Vector_PCB:DIP16, F.Cu at (160.0, 436.9)
- added J_3: LS153A, Star_Wars_Vector_PCB:DIP16, F.Cu at (160.0, 397.5)
- added J_4: LS244A, Star_Wars_Vector_PCB:DIP20, F.Cu at (160.0, 359.4)
- added J_5: LS164A, Star_Wars_Vector_PCB:DIP14, F.Cu at (160.0, 319.4)
- added J_6: LS191_, Star_Wars_Vector_PCB:DIP16, F.Cu at (160.0, 281.3)
- added J_7: PROM, Star_Wars_Vector_PCB:DIP18, F.Cu at (160.0, 244.5)
- added J_9: LS244F, Star_Wars_Vector_PCB:DIP20, F.Cu at (156.2, 160.0)
- added K_2: LS08, Star_Wars_Vector_PCB:DIP14, F.Cu at (139.7, 435.6)
- added K_3: LS153A, Star_Wars_Vector_PCB:DIP16, F.Cu at (139.1, 397.5)
- added K_4: LS244A, Star_Wars_Vector_PCB:DIP20, F.Cu at (139.1, 359.4)
- added K_5: LS164A, Star_Wars_Vector_PCB:DIP14, F.Cu at (139.1, 319.4)
- added K_6: LS08, Star_Wars_Vector_PCB:DIP14, F.Cu at (139.1, 280.0)
- added K_7: PROM, Star_Wars_Vector_PCB:DIP18, F.Cu at (139.1, 244.5)
- added K_8: LS04, Star_Wars_Vector_PCB:DIP14, F.Cu at (139.1, 205.1)
- added K_9: ADC, Star_Wars_Main_PCB:DIP28, F.Cu at (132.1, 160.0)
- added L/M_9: LS259, Star_Wars_Vector_PCB:DIP16, F.Cu at (109.2, 163.8)
- added L_10: 7407, Star_Wars_Vector_PCB:DIP14, F.Cu at (118.7, 113.0)
- added L_2: LS138, Star_Wars_Vector_PCB:DIP16, F.Cu at (116.8, 436.9)
- added L_3: LS157B, Star_Wars_Vector_PCB:DIP16, F.Cu at (118.7, 397.5)
- added L_4: LS374, Star_Wars_Vector_PCB:DIP20, F.Cu at (118.7, 359.4)
- added L_5: LS374, Star_Wars_Vector_PCB:DIP20, F.Cu at (118.7, 319.4)
- added L_6: LS175D, Star_Wars_Vector_PCB:DIP16, F.Cu at (118.7, 281.3)
- added L_7: PROM, Star_Wars_Vector_PCB:DIP18, F.Cu at (118.7, 244.5)
- added L_8: LS138, Star_Wars_Vector_PCB:DIP16, F.Cu at (118.7, 205.1)
- added M_2: LS74, Star_Wars_Vector_PCB:DIP14, F.Cu at (97.2, 436.9)
- added M_3: LS00, Star_Wars_Vector_PCB:DIP14, F.Cu at (98.4, 397.5)
- added M_4: LS374A, Star_Wars_Vector_PCB:DIP20, F.Cu at (98.4, 359.4)
- added M_5: LS374B, Star_Wars_Vector_PCB:DIP20, F.Cu at (98.4, 319.4)
- added M_6: LS83A, Star_Wars_Vector_PCB:DIP16, F.Cu at (98.4, 281.3)
- added M_7: LS299, Star_Wars_Vector_PCB:DIP20, F.Cu at (98.4, 244.5)
- added M_8: LS138, Star_Wars_Vector_PCB:DIP16, F.Cu at (98.4, 205.1)
- added N_11: 082, Star_Wars_Vector_PCB:DIP8, F.Cu at (78.1, 74.3)
- added N_2: LS161, Star_Wars_Vector_PCB:DIP16, F.Cu at (76.8, 436.9)
- added N_3: LS299, Star_Wars_Vector_PCB:DIP20, F.Cu at (77.5, 397.5)
- added N_4: LS83A, Star_Wars_Vector_PCB:DIP16, F.Cu at (77.5, 359.4)
- added N_5: LS83A, Star_Wars_Vector_PCB:DIP16, F.Cu at (77.5, 319.4)
- added N_6: LS83A, Star_Wars_Vector_PCB:DIP16, F.Cu at (77.5, 281.3)
- added N_7: LS138, Star_Wars_Vector_PCB:DIP16, F.Cu at (77.5, 244.5)
- added N_8: LS00, Star_Wars_Vector_PCB:DIP14, F.Cu at (77.5, 205.1)
- added SW1: L_11, Star_Wars_Vector_PCB:DIP8, F.Cu at (115.6, 74.3)
- added SW2: D_10, Star_Wars_Vector_PCB:DIP16, F.Cu at (234.9, 112.4)
- added SW3: E/F_10, Star_Wars_Vector_PCB:DIP16, F.Cu at (214.0, 112.4)

Commit message: Added power traces and components
Parts:
- added C10: .1uf, Star_Wars_Vector_PCB:GenericComp, F.Cu at (179.7, 118.7)
- added C11: .1uf, Star_Wars_Vector_PCB:GenericComp, F.Cu at (179.7, 123.8)
- added C12: .1uf, Star_Wars_Vector_PCB:GenericComp, F.Cu at (179.7, 121.3)
- added C13: .1uf, Star_Wars_Vector_PCB:GenericComp, F.Cu at (160.7, 103.5)
- added C14: .1uf, Star_Wars_Vector_PCB:GenericComp, F.Cu at (160.7, 121.3)
- added C15: .1uf, Star_Wars_Vector_PCB:GenericComp, F.Cu at (160.7, 108.6)
- added C16: .1uf, Star_Wars_Vector_PCB:GenericComp, F.Cu at (160.7, 111.1)
- added C17: .1uf, Star_Wars_Vector_PCB:GenericComp, F.Cu at (160.7, 113.7)
- added C18: .1uf, Star_Wars_Vector_PCB:GenericComp, F.Cu at (160.7, 116.2)
- added C19: .1uf, Star_Wars_Vector_PCB:GenericComp, F.Cu at (160.7, 118.7)
- added C20: .1uf, Star_Wars_Vector_PCB:GenericComp, F.Cu at (160.7, 106.0)
- added C22: .1uf, Star_Wars_Vector_PCB:GenericComp, F.Cu at (273.7, 112.4)
- added C46: .1uf, Star_Wars_Vector_PCB:GenericComp, F.Cu at (139.1, 111.1)
- added C47: .1uf, Star_Wars_Vector_PCB:GenericComp, F.Cu at (139.1, 106.0)
- added C48: .1uf, Star_Wars_Vector_PCB:GenericComp, F.Cu at (139.1, 101.0)
- added C53: .1uf, Star_Wars_Vector_PCB:GenericComp, F.Cu at (136.5, 487.7)
- added C54: .1uf, Star_Wars_Vector_PCB:GenericComp, F.Cu at (184.8, 490.2)
- added C55: .1uf, Star_Wars_Vector_PCB:GenericComp, F.Cu at (268.0, 480.1)
- added C87: .1uf, Star_Wars_Vector_PCB:GenericComp, F.Cu at (189.2, 112.4)
- added C9: .1uf, Star_Wars_Vector_PCB:GenericComp, F.Cu at (179.7, 116.2)
- added C91: .1uf, Star_Wars_Vector_PCB:GenericComp, F.Cu at (85.1, 478.8)
- added C95: .1uf, Star_Wars_Vector_PCB:GenericComp, F.Cu at (241.3, 483.9)
- added C96: .1uf, Star_Wars_Vector_PCB:GenericComp, F.Cu at (243.8, 482.6)
- added CR3: 1N914, Star_Wars_Vector_PCB:GenericComp, F.Cu at (233.7, 482.6)
- added R100: 22k, Star_Wars_Vector_PCB:GenericComp, F.Cu at (236.2, 482.6)
- added R20: 470, Star_Wars_Vector_PCB:GenericComp, F.Cu at (179.7, 103.5)
- added R22: 1k, Star_Wars_Vector_PCB:GenericComp, F.Cu at (179.7, 108.6)
- added R23: 1k, Star_Wars_Vector_PCB:GenericComp, F.Cu at (179.7, 106.0)
- added R24: 1k, Star_Wars_Vector_PCB:GenericComp, F.Cu at (179.7, 111.1)
- added R25: 1k, Star_Wars_Vector_PCB:GenericComp, F.Cu at (179.7, 113.7)
- added R26: 470, Star_Wars_Vector_PCB:GenericComp, F.Cu at (132.1, 79.4)
- added R27: 470, Star_Wars_Vector_PCB:GenericComp, F.Cu at (132.1, 76.8)
- added R28: 470, Star_Wars_Vector_PCB:GenericComp, F.Cu at (132.1, 89.5)
- added R29: 470, Star_Wars_Vector_PCB:GenericComp, F.Cu at (132.1, 71.8)
- added R30: 470, Star_Wars_Vector_PCB:GenericComp, F.Cu at (132.1, 81.9)
- added R31: 470, Star_Wars_Vector_PCB:GenericComp, F.Cu at (132.1, 84.5)
- added R32: 470, Star_Wars_Vector_PCB:GenericComp, F.Cu at (132.1, 87.0)
- added R33: 470, Star_Wars_Vector_PCB:GenericComp, F.Cu at (132.1, 74.3)
- added R34: 1k, Star_Wars_Vector_PCB:GenericComp, F.Cu at (160.7, 71.8)
- added R35: 1k, Star_Wars_Vector_PCB:GenericComp, F.Cu at (160.7, 89.5)
- added R36: 1k, Star_Wars_Vector_PCB:GenericComp, F.Cu at (160.7, 76.8)
- added R37: 1k, Star_Wars_Vector_PCB:GenericComp, F.Cu at (160.7, 79.4)
- added R38: 1k, Star_Wars_Vector_PCB:GenericComp, F.Cu at (160.7, 74.3)
- added R39: 1k, Star_Wars_Vector_PCB:GenericComp, F.Cu at (160.7, 87.0)
- added R40: 1k, Star_Wars_Vector_PCB:GenericComp, F.Cu at (160.7, 84.5)
- added R41: 1k, Star_Wars_Vector_PCB:GenericComp, F.Cu at (160.7, 81.9)
- added R42: 10k, Star_Wars_Vector_PCB:GenericComp, F.Cu at (227.3, 103.5)
- added R43: 10k, Star_Wars_Vector_PCB:GenericComp, F.Cu at (227.3, 106.0)
- added R44: 10k, Star_Wars_Vector_PCB:GenericComp, F.Cu at (227.3, 108.6)
- added R45: 10k, Star_Wars_Vector_PCB:GenericComp, F.Cu at (227.3, 111.1)
- added R46: 10k, Star_Wars_Vector_PCB:GenericComp, F.Cu at (227.3, 113.7)
- added R47: 10k, Star_Wars_Vector_PCB:GenericComp, F.Cu at (227.3, 116.2)
- added R48: 10k, Star_Wars_Vector_PCB:GenericComp, F.Cu at (227.3, 118.7)
- added R49: 10k, Star_Wars_Vector_PCB:GenericComp, F.Cu at (227.3, 121.3)
- added R50: 10k, Star_Wars_Vector_PCB:GenericComp, F.Cu at (198.8, 103.5)
- added R51: 10k, Star_Wars_Vector_PCB:GenericComp, F.Cu at (198.8, 106.0)
- added R52: 10k, Star_Wars_Vector_PCB:GenericComp, F.Cu at (198.8, 108.6)
- added R53: 10k, Star_Wars_Vector_PCB:GenericComp, F.Cu at (198.8, 111.1)
- added R54: 10k, Star_Wars_Vector_PCB:GenericComp, F.Cu at (198.8, 113.7)
- added R55: 10k, Star_Wars_Vector_PCB:GenericComp, F.Cu at (198.8, 116.2)
- added R56: 10k, Star_Wars_Vector_PCB:GenericComp, F.Cu at (198.8, 118.7)
- added R57: 10k, Star_Wars_Vector_PCB:GenericComp, F.Cu at (198.8, 121.3)
- added R59: 10k, Star_Wars_Vector_PCB:GenericComp, F.Cu at (238.8, 483.9)
- added R79: 100, Star_Wars_Vector_PCB:GenericComp, F.Cu at (139.1, 113.7)
- added R80: 100, Star_Wars_Vector_PCB:GenericComp, F.Cu at (139.1, 108.6)
- added R81: 100, Star_Wars_Vector_PCB:GenericComp, F.Cu at (139.1, 103.5)
- added R82: 4.7k, Star_Wars_Vector_PCB:GenericComp, F.Cu at (139.1, 118.7)
- added R83: 4.7k, Star_Wars_Vector_PCB:GenericComp, F.Cu at (139.1, 116.2)
- added R84: 4.7k, Star_Wars_Vector_PCB:GenericComp, F.Cu at (139.1, 121.3)
- added R85: 4.7k, Star_Wars_Vector_PCB:GenericComp, F.Cu at (139.1, 126.4)
- added R86: 4.7k, Star_Wars_Vector_PCB:GenericComp, F.Cu at (139.1, 123.8)
- moved SW2 6.99 mm to (241.9, 112.4)
- moved J20 0.67 mm to (117.8, 37.5)
Connections:
- J18 pad 33: GND -> Net-(J18-Pad33)
- J18 pad 34: Net-(J18-Pad34) -> GND
Routing:
- net GND: track 0.00 -> 2434.2 mm, vias 0 -> 19
- net +5V: track 0.00 -> 2355.6 mm, vias 0 -> 24
- net SPARE1: track 0.00 -> 15.9 mm
- net SLAM: track 0.00 -> 15.9 mm
- net SELF_TEST: track 0.00 -> 15.9 mm
- net R_FIRE: track 0.00 -> 15.9 mm
- net L_FIRE: track 0.00 -> 15.9 mm
- net COIN_R: track 0.00 -> 15.9 mm
- net COIN_L: track 0.00 -> 15.9 mm
- net COIN_AUX: track 0.00 -> 15.9 mm
- net ~SOUNDRST: track 0.00 -> 14.0 mm, vias 0 -> 1
- net ~SOUND: track 0.00 -> 14.0 mm, vias 0 -> 1
- net ~EVMEM: track 0.00 -> 14.0 mm, vias 0 -> 1
- net ~EVGRST: track 0.00 -> 14.0 mm, vias 0 -> 1
- net ~EVGGO: track 0.00 -> 14.0 mm, vias 0 -> 1
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Other:
- board text added: "1"
- board text added: "2"
- board text added: "22"
- board text added: "85"
- board text added: "86"
- board text added: "A"
- board text added: "Z"

Commit message: Added more power traces and components
Parts:
- added TP+10.3UN1: TP, Star_Wars_Vector_PCB:TEST_POINT, F.Cu at (87.0, 73.0)
- added TP+5V2: TP, Star_Wars_Vector_PCB:TEST_POINT, F.Cu at (40.0, 54.6)
- added TPCOINL1: TP, Star_Wars_Vector_PCB:TEST_POINT, F.Cu at (182.2, 84.5)
- added TPCOINR1: TP, Star_Wars_Vector_PCB:TEST_POINT, F.Cu at (172.1, 81.9)
- added TPCOIN_AUX1: TP, Star_Wars_Vector_PCB:TEST_POINT, F.Cu at (172.1, 87.0)
- added TPRST1: TP, Star_Wars_Vector_PCB:TEST_POINT, F.Cu at (39.4, 74.9)
- added TPRST2: TP, Star_Wars_Vector_PCB:TEST_POINT, F.Cu at (43.2, 74.9)
- added TPSELF_TEST1: TP, Star_Wars_Vector_PCB:TEST_POINT, F.Cu at (182.2, 79.4)
- added TPSLAM1: TP, Star_Wars_Vector_PCB:TEST_POINT, F.Cu at (172.1, 74.3)
Routing:
- net GND: track 2434.2 -> 3256.4 mm, vias 19 -> 28
- net +5V: track 2355.6 -> 3045.2 mm, vias 24 -> 32
- net +12V: track 0.00 -> 119.7 mm, vias 0 -> 2
- net +10V: track 0.00 -> 102.1 mm, vias 0 -> 3
- net -5V: track 0.00 -> 73.5 mm, vias 0 -> 1
- net Net-(C18-Pad1): track 0.00 -> 19.0 mm
- net Net-(C16-Pad1): track 0.00 -> 19.0 mm
- net COIN_L: track 15.9 -> 27.4 mm, vias 0 -> 1
- net SLAM: track 15.9 -> 26.8 mm, vias 0 -> 1
- net COIN_AUX: track 15.9 -> 26.1 mm, vias 0 -> 1
- net COIN_CNTR_2: track 0.00 -> 10.2 mm, vias 0 -> 1
- net Net-(C20-Pad1): track 0.00 -> 8.89 mm
- net Net-(C19-Pad1): track 0.00 -> 8.89 mm
- net Net-(C17-Pad1): track 0.00 -> 8.89 mm
- net ~YAW: track 0.00 -> 8.37 mm, vias 0 -> 1
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Other:
- board text added: "+10.3VUN"
- board text added: "+5V2"
- board text added: "COIN"
- board text added: "COINAUX"
- board text added: "COINR"
- board text added: "RESET"
- board text added: "SELFTEST"
- board text added: "SLAM"

Commit message: Added more components
Parts:
- added C4: .1uf, Star_Wars_Vector_PCB:GenericComp, F.Cu at (64.8, 70.5)
- added C49: 100uf 35V, Star_Wars_Vector_PCB:LargeCap, F.Cu at (39.4, 161.3)
- added C50: 100uf 35V, Star_Wars_Vector_PCB:LargeCap, F.Cu at (285.8, 54.0)
- added C51: 100uf 35V, Star_Wars_Vector_PCB:LargeCap, F.Cu at (255.3, 54.0)
- added C7: .1uf, Star_Wars_Vector_PCB:GenericComp, F.Cu at (114.9, 81.3)
- added C8: .1uf, Star_Wars_Vector_PCB:GenericComp, F.Cu at (116.2, 83.8)
- added CR1: 1N914, Star_Wars_Vector_PCB:GenericComp, F.Cu at (38.7, 85.1)
- added Q3: Q_NPN_BCE, Star_Wars_Vector_PCB:VoltReg, F.Cu at (76.2, 94.6)
- added Q4: Q_NPN_BCE, Star_Wars_Vector_PCB:VoltReg, F.Cu at (76.2, 109.2)
- added R12: 10k, Star_Wars_Vector_PCB:GenericComp, F.Cu at (268.0, 410.8)
- added R15: 10k, Star_Wars_Vector_PCB:GenericComp, F.Cu at (236.9, 425.4)
- added R18: 470, Star_Wars_Vector_PCB:GenericComp, F.Cu at (184.8, 76.8)
- added R19: 470, Star_Wars_Vector_PCB:GenericComp, F.Cu at (184.8, 81.9)
- added R21: 470, Star_Wars_Vector_PCB:GenericComp, F.Cu at (184.8, 87.0)
- added R5: 10k, Star_Wars_Vector_PCB:GenericComp, F.Cu at (63.5, 73.0)
- added R6: 100k, Star_Wars_Vector_PCB:GenericComp, F.Cu at (64.8, 78.1)
- added R7: 220, Star_Wars_Vector_PCB:GenericComp, F.Cu at (63.5, 75.6)
- added R8: 15k, Star_Wars_Vector_PCB:GenericComp, F.Cu at (64.8, 80.6)
- added R9: 1k, Star_Wars_Vector_PCB:GenericComp, F.Cu at (64.8, 83.2)
- added TP+12V1: TP, Star_Wars_Vector_PCB:TEST_POINT, F.Cu at (202.6, 54.0)
- added TP+5V1: TP, Star_Wars_Vector_PCB:TEST_POINT, F.Cu at (304.2, 115.6)
- added TP-5V1: TP, Star_Wars_Vector_PCB:TEST_POINT, F.Cu at (231.1, 58.4)
- added TPGND1: TP, Star_Wars_Vector_PCB:TEST_POINT, F.Cu at (299.7, 78.7)
- added TPGND2: TP, Star_Wars_Vector_PCB:TEST_POINT, F.Cu at (40.0, 94.6)
- added VR1: L7805, Star_Wars_Vector_PCB:VoltReg, F.Cu at (266.7, 78.7)
Routing:
- net -5V: track 73.5 -> 320.1 mm, vias 1 -> 2
- net GND: track 3256.4 -> 3451.4 mm, vias 28 -> 30
- net +12V: track 119.7 -> 278.4 mm
- net COIN_CNTR_1: track 0.00 -> 95.3 mm
- net ~HALT: track 8.89 -> 102.5 mm, vias 1 -> 2
- net R~W: track 0.00 -> 78.7 mm, vias 0 -> 1
- net A1: track 0.00 -> 77.5 mm
- net +5V: track 3045.2 -> 3120.4 mm, vias 32 -> 33
- net D1: track 0.00 -> 73.7 mm, vias 0 -> 1
- net A3: track 0.00 -> 72.4 mm
- net A0: track 8.89 -> 81.3 mm
- net D3: track 0.00 -> 68.6 mm, vias 0 -> 1
- net D0: track 8.89 -> 77.5 mm, vias 1 -> 2
- net A2: track 8.89 -> 76.2 mm
- net A5: track 0.00 -> 67.3 mm
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Other:
- board text added: "+"
- board text added: "+12V"
- board text added: "+5V1"
- board text added: "-5V"
- board text added: "GND1"
- board text added: "GND2"
- board text added: "K"

Commit message: Added more power traces
Parts:
- added C69: .1uf, Star_Wars_Vector_PCB:GenericComp, F.Cu at (300.4, 309.9)
- added R11: 10k, Star_Wars_Vector_PCB:GenericComp, F.Cu at (231.8, 275.6)
Connections:
- R_10 pad 1: (no net) -> Net-(R_10-Pad1)
- R_10 pad 14: (no net) -> +5V
- R_10 pad 2: (no net) -> Net-(R_10-Pad2)
- R_10 pad 7: (no net) -> GND
Routing:
- net GND: track 3451.4 -> 5544.1 mm, vias 30 -> 36
- net +5V: track 3120.4 -> 3807.7 mm, vias 33 -> 39

Commit message: Finished the power traces
Parts:
- added C81: .1uf, Star_Wars_Vector_PCB:GenericComp, F.Cu at (300.4, 193.7)
- added C93: 10uf 25V, Star_Wars_Main_PCB:Cap1, F.Cu at (278.1, 78.7)
- added C94: 4.7uf, Star_Wars_Main_PCB:Cap1, F.Cu at (251.5, 457.2)
- moved Q4 0.64 mm to (76.2, 109.9)
Routing:
- net +5V: track 3807.7 -> 5051.7 mm, vias 39 -> 42
- net GND: track 5544.1 -> 5599.6 mm
- net Net-(C94-Pad1): track 2.54 -> 39.4 mm
- net +5EAROM: track 12.7 -> 26.7 mm

Commit message: Added several components
Parts:
- added C21: .1uf, Star_Wars_Vector_PCB:GenericComp, F.Cu at (40.0, 267.3)
- added C52: .1uf, Star_Wars_Vector_PCB:GenericComp, F.Cu at (40.0, 464.2)
- added C56: .1uf, Star_Wars_Vector_PCB:GenericComp, F.Cu at (40.0, 424.2)
- added C59: .1uf, Star_Wars_Vector_PCB:GenericComp, F.Cu at (40.0, 383.5)
- added C62: .1uf, Star_Wars_Vector_PCB:GenericComp, F.Cu at (40.0, 345.4)
- added C65: .1uf, Star_Wars_Vector_PCB:GenericComp, F.Cu at (306.7, 351.2)
- added C66: .1uf, Star_Wars_Vector_PCB:GenericComp, F.Cu at (40.0, 305.4)
- added C73: .1uf, Star_Wars_Vector_PCB:GenericComp, F.Cu at (300.4, 267.3)
- added C74: .1uf, Star_Wars_Vector_PCB:GenericComp, F.Cu at (40.0, 230.5)
- added C77: .1uf, Star_Wars_Vector_PCB:GenericComp, F.Cu at (300.4, 230.5)
- added C78: .1uf, Star_Wars_Vector_PCB:GenericComp, F.Cu at (40.0, 191.1)
- added C82: .1uf, Star_Wars_Vector_PCB:GenericComp, F.Cu at (40.0, 144.8)
- added C83: .1uf, Star_Wars_Vector_PCB:GenericComp, F.Cu at (97.8, 163.2)
- added C85: .1uf, Star_Wars_Vector_PCB:GenericComp, F.Cu at (300.4, 147.3)
- added C86: .1uf, Star_Wars_Vector_PCB:GenericComp, F.Cu at (46.4, 113.0)
- added CR2: BLUE, Star_Wars_Vector_PCB:LED, F.Cu at (55.2, 170.2)
- added CR4: BLUE LED, Star_Wars_Vector_PCB:LED, F.Cu at (95.2, 132.1)
- added CR5: BLUE LED, Star_Wars_Vector_PCB:LED, F.Cu at (95.2, 119.4)
- added CR6: BLUE LED, Star_Wars_Vector_PCB:LED, F.Cu at (95.2, 105.4)
- added R13: 1k, Star_Wars_Vector_PCB:GenericComp, F.Cu at (94.0, 163.2)
- added R14: 1k, Star_Wars_Vector_PCB:GenericComp, F.Cu at (91.4, 163.2)
- added R16: 1k, Star_Wars_Vector_PCB:GenericComp, F.Cu at (105.4, 111.8)
- added R17: 1k, Star_Wars_Vector_PCB:GenericComp, F.Cu at (102.9, 111.8)
- added R58: 1k, Star_Wars_Vector_PCB:GenericComp, F.Cu at (88.9, 163.2)
Routing:
- net +5V: track 5051.7 -> 5159.0 mm, vias 42 -> 41
- net GND: track 5599.6 -> 5692.3 mm
