File: pcb/star_wars_arcade_main_pcb.kicad_pcb (KiCad board)
At the start: 2 copper layers, 292.1 x 525.8 mm, 254 parts, among them J17 Main_Connector, J18 Cat_Box_Conn, J20 J20, Q3 Q_NPN_BCE, Q4 Q_NPN_BCE, SW1 L_11, SW2 D_10, SW3 E/F_10

Commit message: Added more components
Parts:
- added C1: .1uf, Star_Wars_Vector_PCB:GenericComp, F.Cu at (59.1, 469.3)
- added C2: 100pf, Star_Wars_Vector_PCB:CapBrown, F.Cu at (66.7, 489.6)
- added C23: .1uf, Star_Wars_Vector_PCB:GenericComp, F.Cu at (-14.0, 390.5)
- added C24: .1uf, Star_Wars_Vector_PCB:GenericComp, F.Cu at (69.2, 474.3)
- added C3: 39pf, Star_Wars_Vector_PCB:CapBrown, F.Cu at (41.9, 478.8)
- added C45: .1uf, Star_Wars_Vector_PCB:GenericComp, F.Cu at (-22.8, 372.4)
- added C5: .1uf, Star_Wars_Vector_PCB:GenericComp, F.Cu at (241.9, 450.2)
- added C57: .1uf, Star_Wars_Vector_PCB:GenericComp, F.Cu at (-19.9, 372.4)
- added C58: .1uf, Star_Wars_Vector_PCB:GenericComp, F.Cu at (-17.0, 372.4)
- added C60: .1uf, Star_Wars_Vector_PCB:GenericComp, F.Cu at (-14.1, 372.4)
- added C61: .1uf, Star_Wars_Vector_PCB:GenericComp, F.Cu at (-11.2, 372.4)
- added C63: .1uf, Star_Wars_Vector_PCB:GenericComp, F.Cu at (-8.32, 372.4)
- added C64: .1uf, Star_Wars_Vector_PCB:GenericComp, F.Cu at (-5.42, 372.4)
- added C67: .1uf, Star_Wars_Vector_PCB:GenericComp, F.Cu at (-2.52, 372.4)
- added C68: .1uf, Star_Wars_Vector_PCB:GenericComp, F.Cu at (0.38, 372.4)
- added C70: .1uf, Star_Wars_Vector_PCB:GenericComp, F.Cu at (-11.0, 390.6)
- added C71: .1uf, Star_Wars_Vector_PCB:GenericComp, F.Cu at (-25.7, 372.4)
- added C72: .1uf, Star_Wars_Vector_PCB:GenericComp, F.Cu at (-8.13, 390.6)
- added C75: .1uf, Star_Wars_Vector_PCB:GenericComp, F.Cu at (-5.23, 390.6)
- added C76: .1uf, Star_Wars_Vector_PCB:GenericComp, F.Cu at (-2.33, 390.6)
- added C79: .1uf, Star_Wars_Vector_PCB:GenericComp, F.Cu at (0.57, 390.6)
- added C80: .1uf, Star_Wars_Vector_PCB:GenericComp, F.Cu at (3.28, 372.4)
- added C84: .1uf, Star_Wars_Vector_PCB:GenericComp, F.Cu at (3.47, 390.6)
- added C88: .1uf, Star_Wars_Vector_PCB:GenericComp, F.Cu at (6.18, 372.4)
- added C89: .1uf, Star_Wars_Vector_PCB:GenericComp, F.Cu at (6.37, 390.6)
- added C90: .1uf, Star_Wars_Vector_PCB:GenericComp, F.Cu at (9.08, 372.4)
- added C92: .1uf, Star_Wars_Vector_PCB:GenericComp, F.Cu at (9.27, 390.6)
- added J16: Aud_Conn, Star_Wars_Main_PCB:Aud_Con, F.Cu at (65.3, 139.1)
- added L1: 100uH, Star_Wars_Main_PCB:Ind, F.Cu at (41.9, 474.3)
- added Q1: 2N3904, Star_Wars_Vector_PCB:GenericTrans, F.Cu at (58.4, 475.0)
- added R1: 10k, Star_Wars_Vector_PCB:GenericComp, F.Cu at (43.2, 491.5)
- added R10: 1k, Star_Wars_Vector_PCB:GenericComp, F.Cu at (240.7, 452.8)
- added R2: 10k, Star_Wars_Vector_PCB:GenericComp, F.Cu at (40.0, 490.2)
- added R3: 68, Star_Wars_Vector_PCB:GenericComp, F.Cu at (41.9, 470.5)
- added R4: 1k, Star_Wars_Vector_PCB:GenericComp, F.Cu at (233.0, 316.9)
- added R91: 1k, Star_Wars_Vector_PCB:GenericComp, F.Cu at (54.6, 154.9)
- added R92: 1k, Star_Wars_Vector_PCB:GenericComp, F.Cu at (231.8, 158.8)
- added R93: 1k, Star_Wars_Vector_PCB:GenericComp, F.Cu at (169.5, 201.9)
- added R94: 1k, Star_Wars_Vector_PCB:GenericComp, F.Cu at (127.6, 201.9)
- added R95: 1k, Star_Wars_Vector_PCB:GenericComp, F.Cu at (64.8, 203.8)
- added R96: 1k, Star_Wars_Vector_PCB:GenericComp, F.Cu at (47.6, 398.8)
- added R97: 1k, Star_Wars_Vector_PCB:GenericComp, F.Cu at (68.6, 201.3)
- added TP+5V3: TP, Star_Wars_Vector_PCB:TEST_POINT, F.Cu at (290.8, 535.3)
- added TP+5V4: TP, Star_Wars_Vector_PCB:TEST_POINT, F.Cu at (52.1, 500.4)
- added TP3MHZ1: TP, Star_Wars_Vector_PCB:TEST_POINT, F.Cu at (88.9, 462.3)
- added TP6MHZ1: TP, Star_Wars_Vector_PCB:TEST_POINT, F.Cu at (77.5, 422.9)
- added TPCATSTR1: TP, Star_Wars_Vector_PCB:TEST_POINT, F.Cu at (280.0, 414.7)
- added TPDIAGN1: TP, Star_Wars_Vector_PCB:TEST_POINT, F.Cu at (170.8, 143.5)
- added TPE1: TP, Star_Wars_Vector_PCB:TEST_POINT, F.Cu at (258.4, 396.2)
- added TPEVMEM1: TP, Star_Wars_Vector_PCB:TEST_POINT, F.Cu at (107.3, 454.7)
- added TPFIRE/START1: TP, Star_Wars_Vector_PCB:TEST_POINT, F.Cu at (156.2, 143.5)
- added TPGND3: TP, Star_Wars_Vector_PCB:TEST_POINT, F.Cu at (301.6, 514.4)
- added TPGND4: TP, Star_Wars_Vector_PCB:TEST_POINT, F.Cu at (38.7, 514.4)
- added TPHALT1: TP, Star_Wars_Vector_PCB:TEST_POINT, F.Cu at (234.9, 456.6)
- added TPMPAGE1: TP, Star_Wars_Vector_PCB:TEST_POINT, F.Cu at (109.2, 189.9)
- added TPQ1: TP, Star_Wars_Vector_PCB:TEST_POINT, F.Cu at (258.4, 389.9)
- added TPRESET1: TP, Star_Wars_Vector_PCB:TEST_POINT, F.Cu at (108.0, 143.5)
- added TPROM0: TP, Star_Wars_Vector_PCB:TEST_POINT, F.Cu at (278.8, 459.7)
- added TPROM1: TP, Star_Wars_Vector_PCB:TEST_POINT, F.Cu at (278.8, 455.3)
- added TPROM2: TP, Star_Wars_Vector_PCB:TEST_POINT, F.Cu at (278.8, 450.9)
- added TPROM3: TP, Star_Wars_Vector_PCB:TEST_POINT, F.Cu at (278.8, 464.2)
- added TPROM4: TP, Star_Wars_Vector_PCB:TEST_POINT, F.Cu at (102.2, 462.9)
- added TPRW1: TP, Star_Wars_Vector_PCB:TEST_POINT, F.Cu at (258.4, 402.6)
- added TPRWB1: TP, Star_Wars_Vector_PCB:TEST_POINT, F.Cu at (215.9, 342.9)
- added TPWDDIS1: TP, Star_Wars_Vector_PCB:TEST_POINT, F.Cu at (228.6, 301.6)
- added Y1: 12.096MHz, Star_Wars_Main_PCB:Y, F.Cu at (53.3, 480.7)
Routing:
- net GND: track 5692.3 -> 5778.7 mm
- net +5V: track 5159.0 -> 5223.7 mm
- net Net-(C2-Pad2): track 0.00 -> 16.5 mm
- net P93: track 0.00 -> 8.89 mm
- net Net-(CR2-Pad2): track 0.00 -> 8.26 mm
- net P92: track 0.00 -> 5.72 mm
- net ~ROM4: track 0.00 -> 5.08 mm
- net ~HALT: track 102.1 -> 107.2 mm
- net R~W: track 78.7 -> 83.8 mm
- net Net-(C_2-Pad34): track 0.00 -> 5.08 mm
- net Net-(C13-Pad1): track 0.00 -> 5.08 mm
- net ECLKQ: track 14.0 -> 19.1 mm
- net ~RESET: track 8.25 -> 13.3 mm
- net ~PCLR: track 0.00 -> 5.08 mm
- net ~EVMEM: track 14.0 -> 19.1 mm
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Other:
- board text added: "+5V3"
- board text added: "+5V4"
- board text added: "3MHZ"
- board text added: "6MHZ"
- board text added: "DIAGN"
- board text added: "ECLKQ"
- board text added: "ETEST"
- board text added: "FIRE/ST"
- board text added: "GND3"
- board text added: "GND4"
- board text added: "HALT"
- board text added: "J17"
- board text added: "MPAGE"
- board text added: "R/W-B"
- board text added: "WDDIS"
- board text added: "~R/W"
- board text added: "~RESET"
- board text added: "~ROM0"
- board text added: "~ROM1"
- board text added: "~ROM2"
- board text added: "~ROM3"
- board text added: "~ROM4"
- board text added: "~VMEM"
