File: pcb/star_wars_arcade_main_pcb.kicad_pcb (KiCad board)
At the start: 2 copper layers, 292.1 x 525.8 mm, 320 parts, among them J16 Aud_Conn, J17 Main_Connector, J18 Cat_Box_Conn, J20 J20, Q1 2N3904, Q3 Q_NPN_BCE, Q4 Q_NPN_BCE, SW1 L_11, SW2 D_10, SW3 E/F_10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

Commit message: Finished placing all components
Parts:
- moved C88 326.1 mm to (251.5, 157.5), turned to 180 degrees
- moved C84 295.1 mm to (186.1, 158.8), turned to 180 degrees
- moved C90 277.5 mm to (230.5, 205.1), turned to 180 degrees
- moved C89 275.6 mm to (210.2, 205.1), turned to 180 degrees
- moved C45 269.5 mm to (145.4, 161.9), turned to 180 degrees
- moved C92 252.0 mm to (243.8, 482.6), turned to 180 degrees
- moved C23 250.5 mm to (210.2, 278.8), turned to 180 degrees
- moved C80 249.7 mm to (189.2, 205.7), turned to 180 degrees
- moved C76 242.4 mm to (191.1, 244.5), turned to 180 degrees
- moved C70 234.0 mm to (47.0, 163.8), turned to 180 degrees
- moved C72 225.6 mm to (189.2, 281.3), turned to 180 degrees
- moved C79 204.3 mm to (87.6, 205.7), turned to 180 degrees
- moved C61 203.3 mm to (190.5, 397.5), turned to 180 degrees
- moved C58 200.2 mm to (172.1, 438.1), turned to 180 degrees
- moved C68 199.1 mm to (191.8, 317.5), turned to 180 degrees
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Routing:
- net GND: track 5778.7 -> 5917.5 mm, vias 36 -> 39
- net +5V: track 5223.7 -> 5351.9 mm, vias 41 -> 49

Commit message: Added mounting holes
Parts:
- added REF**: MountingHole, Star_Wars_Vector_PCB:MountingHole, F.Cu at (299.7, 353.1)
- added REF**: MountingHole, Star_Wars_Vector_PCB:MountingHole, F.Cu at (43.2, 361.3)
Routing:
- net +5V: track 5351.9 -> 5352.6 mm
Changed lines of the file:
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@@
     (tracks 1884)
     (zones 0)
-    (modules 320)
+    (modules 322)
     (nets 622)
   )
@@
     (mod_text_size 1 1)
     (mod_text_width 0.15)
-    (pad_size 1.905 1.905)
-    (pad_drill 1.016)
+    (pad_size 4.826 4.826)
+    (pad_drill 4.572)
     (pad_to_mask_clearance 0.051)
     (solder_mask_min_width 0.25)
@@
   )
   (module Star_Wars_Vector_PCB:MountingHole (layer F.Cu)
+    (at 299.72 353.06)
+    (fp_text reference REF** (at 0 3.81) (layer F.SilkS) hide
+      (effects (font (size 1 1) (thickness 0.15)))
+    )
+    (fp_text value MountingHole (at 0 -3.81) (layer F.Fab)
+      (effects (font (size 1 1) (thickness 0.15)))
+    )
+    (pad 1 thru_hole circle (at 0 0) (size 4.826 4.826) (drill 4.572) (layers *.Cu *.Mask))
+  )
+  (module Star_Wars_Vector_PCB:MountingHole (layer F.Cu)
+    (at 43.18 361.315)
+    (fp_text reference REF** (at 0 3.81) (layer F.SilkS) hide
+      (effects (font (size 1 1) (thickness 0.15)))
+    )
+    (fp_text value MountingHole (at 0 -3.81) (layer F.Fab)
+      (effects (font (size 1 1) (thickness 0.15)))
+    )
+    (pad 1 thru_hole circle (at 0 0) (size 4.826 4.826) (drill 4.572) (layers *.Cu *.Mask))
+  )
+  (module Star_Wars_Vector_PCB:MountingHole (layer F.Cu)
     (at 311.15 39.37)
     (fp_text reference REF** (at 0 3.81) (layer F.SilkS) hide
@@
   (via (at 33.655 386.715) (size 1.524) (drill 1.016) (layers F.Cu B.Cu) (net 1))
   (via (at 33.655 427.355) (size 1.524) (drill 1.016) (layers F.Cu B.Cu) (net 1))
-  (via (at 33.655 467.36) (size 1.524) (drill 1.016) (layers F.Cu B.Cu) (net 1))
   (via (at 298.45 45.085) (size 2.286) (drill 1.016) (layers F.Cu B.Cu) (net 1))
   (via (at 37.465 59.055) (size 2.286) (drill 1.016) (layers F.Cu B.Cu) (net 1))
@@
   (segment (start 290.195 412.115) (end 290.195 412.115) (width 1.524) (layer F.Cu) (net 1))
   (via (at 290.195 412.115) (size 1.524) (drill 1.016) (layers F.Cu B.Cu) (net 1))
-  (segment (start 33.655 467.36) (end 28.575 467.36) (width 1.524) (layer B.Cu) (net 1))
-  (segment (start 64.135 467.36) (end 64.135 469.265) (width 1.524) (layer F.Cu) (net 1))
   (segment (start 85.09 466.725) (end 85.09 469.265) (width 1.524) (layer F.Cu) (net 1))
   (segment (start 85.09 469.265) (end 85.09 473.71) (width 1.524) (layer F.Cu) (net 1))
@@
   (segment (start 200.025 422.275) (end 215.9 422.275) (width 1.524) (layer F.Cu) (net 1))
   (segment (start 215.9 422.275) (end 243.205 422.275) (width 1.524) (layer F.Cu) (net 1))
-  (segment (start 45.085 464.185) (end 45.085 467.36) (width 1.524) (layer F.Cu) (net 1))
-  (segment (start 33.655 467.36) (end 45.085 467.36) (width 1.524) (layer F.Cu) (net 1))
   (segment (start 45.085 383.54) (end 45.085 387.985) (width 1.524) (layer F.Cu) (net 1))
   (segment (start 45.085 387.985) (end 41.275 387.985) (width 1.524) (layer F.Cu) (net 1))
@@
   (segment (start 60.96 387.985) (end 47.625 387.985) (width 1.524) (layer F.Cu) (net 1))
   (segment (start 47.625 387.985) (end 45.085 387.985) (width 1.524) (layer F.Cu) (net 1))
-  (segment (start 55.88 474.98) (end 55.88 467.36) (width 1.524) (layer F.Cu) (net 1))
-  (segment (start 45.085 467.36) (end 55.88 467.36) (width 1.524) (layer F.Cu) (net 1))
-  (segment (start 55.88 467.36) (end 64.135 467.36) (width 1.524) (layer F.Cu) (net 1))
   (segment (start 231.775 152.4) (end 231.775 149.225) (width 1.524) (layer F.Cu) (net 1))
   (segment (start 64.77 197.485) (end 64.77 195.58) (width 1.524) (layer F.Cu) (net 1))
@@
   (via (at 172.085 426.085) (size 1.524) (drill 1.016) (layers F.Cu B.Cu) (net 1))
   (segment (start 172.085 433.07) (end 172.085 426.085) (width 1.524) (layer B.Cu) (net 1))
+  (segment (start 64.135 466.725) (end 64.135 469.265) (width 1.524) (layer F.Cu) (net 1))
+  (segment (start 55.88 466.725) (end 64.135 466.725) (width 1.524) (layer F.Cu) (net 1))
+  (segment (start 55.88 466.725) (end 55.88 474.98) (width 1.524) (layer F.Cu) (net 1))
+  (segment (start 45.085 464.185) (end 45.085 466.725) (width 1.524) (layer F.Cu) (net 1))
+  (segment (start 45.085 466.725) (end 55.88 466.725) (width 1.524) (layer F.Cu) (net 1))
+  (segment (start 33.655 466.725) (end 28.575 466.725) (width 1.524) (layer B.Cu) (net 1))
+  (via (at 33.655 466.725) (size 1.524) (drill 1.016) (layers F.Cu B.Cu) (net 1))
+  (segment (start 33.655 466.725) (end 45.085 466.725) (width 1.524) (layer F.Cu) (net 1))
   (via (at 85.725 292.735) (size 1.524) (drill 1.016) (layers F.Cu B.Cu) (net 2))
   (via (at 108.585 292.735) (size 1.524) (drill 1.016) (layers F.Cu B.Cu) (net 2))

Commit message: Started adding signal traces
Parts:
- moved C92 1.42 mm to (244.5, 481.3)
- moved CR3 1.42 mm to (234.3, 481.3)
- moved R100 1.42 mm to (236.9, 481.3)
- moved R59 1.42 mm to (239.4, 482.6)
- moved C95 1.42 mm to (241.9, 482.6)
- moved D/E0 0.64 mm to (231.8, 512.4)
- moved E_1 0.63 mm to (224.8, 479.4)
Routing:
- net AB3: track 14.0 -> 391.7 mm, vias 1 -> 4
- net AB4: track 14.0 -> 367.9 mm, vias 1 -> 4
- net AB2: track 14.0 -> 335.5 mm, vias 1 -> 2
- net AB1: track 14.0 -> 333.4 mm, vias 1 -> 2
- net AB0: track 14.0 -> 332.1 mm, vias 1 -> 6
- net AB5: track 14.0 -> 324.5 mm
- net AB7: track 14.0 -> 320.7 mm, vias 1 -> 2
- net AB12: track 14.0 -> 318.1 mm, vias 1 -> 4
- net AB6: track 14.0 -> 312.0 mm, vias 1 -> 3
- net AB11: track 14.0 -> 277.5 mm
- net AB8: track 14.0 -> 271.1 mm
- net AB10: track 14.0 -> 264.8 mm
- net P92: track 5.72 -> 220.0 mm, vias 0 -> 2
- net R~W~B: track 19.1 -> 225.7 mm, vias 1 -> 3
- net GND: track 5917.5 -> 6117.9 mm, vias 39 -> 45
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Other:
- board text added: "CATSTR"

Commit message: Added more signal traces
Parts:
- moved R82 1.27 mm to (137.8, 118.7), turned to 270 degrees
- moved R83 1.27 mm to (137.8, 116.2), turned to 270 degrees
Routing:
- net AB1: track 333.4 -> 553.1 mm, vias 2 -> 4
- net AB6: track 312.0 -> 518.7 mm, vias 3 -> 5
- net AB0: track 332.1 -> 514.3 mm, vias 6 -> 8
- net AB2: track 335.5 -> 504.5 mm, vias 2 -> 4
- net IP0: track 0.00 -> 165.7 mm, vias 0 -> 1
- net IP5: track 0.00 -> 153.7 mm, vias 0 -> 1
- net ~SOUND: track 172.7 -> 314.3 mm, vias 2 -> 3
- net ~DVDDH: track 0.00 -> 120.3 mm, vias 0 -> 2
- net CIG*: track 0.00 -> 102.9 mm, vias 0 -> 2
- net DB0: track 0.00 -> 96.5 mm, vias 0 -> 1
- net MA0: track 0.00 -> 90.1 mm, vias 0 -> 2
- net ~SOUNDRST: track 28.2 -> 93.0 mm, vias 3 -> 4
- net GND: track 6117.9 -> 6182.7 mm, vias 45 -> 47
- net Net-(K_4-Pad8): track 0.00 -> 56.5 mm
- net +5V: track 5391.3 -> 5444.6 mm
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
Commit message: Added more signal traces, 951 disconnected signals remain
Parts:
- moved C68 0.63 mm to (191.8, 318.1)
- moved C94 0.63 mm to (251.5, 457.8)
- moved F_5 0.63 mm to (204.5, 317.5)
- moved H_5 0.63 mm to (177.8, 317.5)
- moved TPHALT1 0.63 mm to (234.9, 457.2)
Routing:
- net +5EAROM: track 40.3 -> 531.1 mm, vias 1 -> 3
- net VGHALT: track 87.6 -> 457.2 mm, vias 2 -> 4
- net GND: track 6182.7 -> 6536.4 mm, vias 47 -> 51
- net ~EVGGO: track 73.5 -> 389.1 mm, vias 3 -> 4
- net AB5: track 324.5 -> 563.5 mm, vias 1 -> 4
- net Net-(D/E0-Pad19): track 84.7 -> 323.5 mm
- net ~SOUNDRST: track 93.0 -> 321.6 mm, vias 4 -> 5
- net Net-(J_2-Pad15): track 0.00 -> 212.1 mm, vias 0 -> 1
- net ~MW1: track 0.00 -> 199.5 mm, vias 0 -> 3
- net P94: track 0.00 -> 198.1 mm, vias 0 -> 3
- net ~NSTORE: track 0.00 -> 196.2 mm, vias 0 -> 1
- net S2: track 0.00 -> 196.1 mm, vias 0 -> 1
- net IP2: track 12.1 -> 187.9 mm, vias 1 -> 2
- net ~MBCON: track 0.00 -> 174.6 mm, vias 0 -> 1
- net IP4: track 0.00 -> 162.6 mm, vias 0 -> 1
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
Commit message: 891 unconnected signal remain
Parts:
- moved R4 0.63 mm to (232.4, 316.9)
Connections:
- D_3 pad 1: Net-(D_3-Pad1) -> GND
- D_3 pad 10: Net-(D_3-Pad10) -> GND
- D_3 pad 14: ~INCBIC -> Net-(D_3-Pad14)
- D_3 pad 4: Net-(D_3-Pad4) -> GND
- D_3 pad 9: Net-(D_3-Pad9) -> GND
- F_3 pad 13: Net-(D_3-Pad4) -> Net-(D_3-Pad14)
Routing:
- net 3MHZ: track 5.08 -> 260.4 mm, vias 0 -> 2
- net Net-(B/C_0-Pad14): track 19.0 -> 235.2 mm, vias 1 -> 2
- net Net-(B/C_0-Pad15): track 24.1 -> 238.1 mm, vias 1 -> 2
- net Net-(E_1-Pad10): track 12.7 -> 188.6 mm, vias 0 -> 1
- net ~RESET: track 133.6 -> 308.9 mm, vias 3 -> 4
- net D1: track 73.7 -> 241.9 mm, vias 1 -> 3
- net P92: track 220.0 -> 387.0 mm, vias 2 -> 3
- net D7: track 160.5 -> 314.2 mm, vias 2 -> 3
- net D2: track 130.2 -> 261.6 mm, vias 3 -> 5
- net 1.5MHZ: track 0.00 -> 119.1 mm, vias 0 -> 1
- net A14: track 49.5 -> 158.1 mm
- net D0: track 159.9 -> 266.6 mm, vias 3 -> 4
- net A15: track 52.1 -> 156.8 mm
- net MDB2: track 40.6 -> 141.0 mm, vias 1 -> 3
- net AB12: track 318.1 -> 407.3 mm
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
Commit message: Added more signal traces
Parts:
- moved CR4 0.64 mm to (94.6, 132.1)
- moved CR5 0.64 mm to (94.6, 119.4)
- moved CR6 0.64 mm to (94.6, 105.4)
- moved R14 0.64 mm to (92.1, 163.2)
- moved R13 0.63 mm to (94.6, 163.2)
- moved R58 0.63 mm to (89.5, 163.2)
Connections:
- N_11 pad 5: GND -> Net-(N_11-Pad5)
- N_11 pad 6: GND -> Net-(N_11-Pad6)
- R16 pad 1: Net-(L/M_9-Pad4) -> Net-(L_10-Pad6)
- R17 pad 1: Net-(L/M_9-Pad5) -> Net-(L_10-Pad4)
Routing:
- net GND: track 6598.0 -> 7303.6 mm, vias 52 -> 58
- net Net-(P_2-Pad12): track 10.2 -> 349.9 mm
- net 12MHZ: track 0.00 -> 223.5 mm, vias 0 -> 4
- net S1: track 12.1 -> 162.3 mm, vias 1 -> 2
- net LED1: track 0.00 -> 130.4 mm
- net +12V: track 278.4 -> 403.6 mm, vias 2 -> 4
- net -5V: track 320.1 -> 441.0 mm, vias 2 -> 4
- net ~PCLR: track 19.0 -> 134.6 mm, vias 1 -> 2
- net D3: track 163.2 -> 265.1 mm, vias 2 -> 4
- net +5V: track 5518.3 -> 5617.3 mm, vias 49 -> 51
- net 750KHZ: track 77.5 -> 174.6 mm, vias 0 -> 1
- net P92: track 387.0 -> 472.1 mm
- net COIN_CNTR_2: track 50.2 -> 134.0 mm, vias 1 -> 2
- net Net-(E_9-Pad11): track 4.44 -> 86.4 mm
- net Net-(E_9-Pad13): track 4.44 -> 83.8 mm
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
Commit message: Added more signal traces
Parts:
- moved TPRWB1 0.64 mm to (215.9, 343.5)
- moved C61 0.63 mm to (189.9, 397.5)
- moved C90 0.63 mm to (229.9, 205.1)
- moved D_7 0.63 mm to (241.9, 244.5)
- moved R11 0.63 mm to (232.4, 275.6)
- moved R4 0.63 mm to (233.0, 316.9)
Connections:
- E_6 pad 1: S1 -> IP7
- E_6 pad 2: IP7 -> S1
- F_3 pad 14: ~INCBIC -> Net-(E_3-Pad13)
- F_3 pad 4: Net-(E_3-Pad13) -> GND
- J16 pad 8: S1 -> S1_
- J16 pad 9: S2 -> S2_
- J20 pad 5: S1 -> S1_
- J20 pad 8: S2 -> S2_
Routing:
- net MPAGE: track 19.7 -> 465.5 mm, vias 1 -> 4
- net Net-(E_1-Pad10): track 188.6 -> 559.1 mm, vias 1 -> 2
- net D7: track 331.4 -> 575.2 mm, vias 4 -> 6
- net GND: track 7303.6 -> 7544.9 mm, vias 58 -> 59
- net D0: track 324.4 -> 565.7 mm, vias 5 -> 6
- net D6: track 248.9 -> 471.2 mm, vias 3 -> 4
- net D5: track 205.1 -> 426.1 mm, vias 2 -> 4
- net D3: track 265.1 -> 484.8 mm, vias 4 -> 5
- net ~WE: track 78.7 -> 294.0 mm, vias 2 -> 3
- net D4: track 243.8 -> 445.8 mm
- net S2_: track 0.00 -> 196.1 mm, vias 0 -> 1
- net 1.5MHZ: track 119.1 -> 314.9 mm, vias 1 -> 5
- net ~INCBIC: track 0.00 -> 160.9 mm, vias 0 -> 2
- net S1_: track 0.00 -> 150.2 mm, vias 0 -> 1
- net ~CLEAR_ACC: track 0.00 -> 123.3 mm, vias 0 -> 2
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